File: PCIEX4.kicad_sch (KiCad schematic)
At the start: 0 parts

Commit message: finished schematic draft and started placing components
Parts:
- added C1078, C1079, C1080, C1081, C1082, C1083, C2, C3: 220nF/16V, A_HDJ_Library:C_0402_1005Metric, symbol Device:C_Small
- added C1084, C1085, C1088, C15: 100nF/16V, A_HDJ_Library:C_0402_1005Metric, symbol Device:C
- added C1086, C1087: 100uF/25V, A_HDJ_Library:CP_Elec_6.3x7.7, symbol Device:C_Polarized
- added C14: 10uF/10V, A_HDJ_Library:C_0402_1005Metric, symbol Device:C
- added C16: 470uF/6.3V, A_HDJ_Library:CP_Elec_6.3x7.7, symbol Device:C_Polarized
- added J1006: Bus_PCI_Express_x4, A_HDJ_Library:PCIe_x4_Gen3Slot_Connectors, symbol Connector:Bus_PCI_Express_x4
- added TP1006: TestPoint, A_HDJ_Library:TestPoint_Pad_D1.5mm, symbol Connector:TestPoint
Connections:
- new net +12VA: C1084.1, C1085.1, C1086.1, C1087.1, J1006.A2 (+12V), J1006.A3 (+12V), J1006.B1 (+12V), J1006.B2 (+12V), J1006.B3 (+12V)
- new net +3V3: C1088.2, C14.2, C15.1, C16.1, J1006.A10 (+3.3V), J1006.A9 (+3.3V), J1006.B10 (3.3Vaux), J1006.B8 (+3.3V)
- new net GND: C1084.2, C1085.2, C1086.2, C1087.2, C1088.1, C14.1, C15.2, C16.2, J1006.A1 (~{PRSNT1}), J1006.A12 (GND), J1006.A15 (GND), J1006.A18 (GND), J1006.A20 (GND), J1006.A23 (GND), J1006.A24 (GND), J1006.A27 (GND), J1006.A28 (GND), J1006.A31 (GND), J1006.A4 (GND), J1006.B13 (GND), J1006.B16 (GND), J1006.B17 (~{PRSNT2}), J1006.B18 (GND), J1006.B21 (GND), J1006.B22 (GND), J1006.B25 (GND), J1006.B26 (GND), J1006.B29 (GND), J1006.B31 (~{PRSNT2}), J1006.B32 (GND), J1006.B4 (GND), J1006.B7 (GND)
- new net PCIE30_TX0_N: C2.2, J1006.B15 (PETn0)
- new net PCIE30_TX0_P: C1078.2, J1006.B14 (PETp0)
- new net PCIE30_TX1_N: C1079.2, J1006.B20 (PETn1)
- new net PCIE30_TX1_P: C3.2, J1006.B19 (PETp1)
- new net PCIE30_TX2_N: C1081.2, J1006.B24 (PETn2)
- new net PCIE30_TX2_P: C1080.2, J1006.B23 (PETp2)
- new net PCIE30_TX3_N: C1083.2, J1006.B28 (PETn3)
- new net PCIE30_TX3_P: C1082.2, J1006.B27 (PETp3)
- new net PCIE_RX_0+: J1006.A16 (PERp0)
- new net PCIE_RX_0-: J1006.A17 (PERn0)
- new net PCIE_RX_1+: J1006.A21 (PERp1)
- new net PCIE_RX_1-: J1006.A22 (PERn1)
- new net PCIE_RX_2+: J1006.A25 (PERp2)
- new net PCIE_RX_2-: J1006.A26 (PERn2)
- new net PCIE_RX_3+: J1006.A29 (PERp3)
- new net PCIE_RX_3-: J1006.A30 (PERn3)
- new net PCIE_TX_0+: C1078.1
- new net PCIE_TX_0-: C2.1
- new net PCIE_TX_1+: C3.1
- new net PCIE_TX_1-: C1079.1
- new net PCIE_TX_2+: C1080.1
- new net PCIE_TX_2-: C1081.1
- new net PCIE_TX_3+: C1082.1
- new net PCIE_TX_3-: C1083.1
- new net REFCLK+: J1006.A13 (REFCLK+)
- new net REFCLK-: J1006.A14 (REFCLK-)
- new net ~{PLT_RST}: J1006.A11 (~{PERST}), TP1006.1
- new net ~{WAKE}: J1006.B11 (~{WAKE})
- no-connect marks 0 -> 11

Commit message: commit before removing duplicated glasgow
Parts:
- removed C1078, C2: 220nF/16V, A_HDJ_Library:C_0402_1005Metric, symbol Device:C_Small
- renumbered C3 to C51, C1079 to C52, C1080 to C53, C1081 to C54, C1082 to C55, C1083 to C56, C1084 to C57, C1085 to C58, C1086 to C59, C1087 to C60, C1088 to C61, C14 to C62, C15 to C63, C16 to C64, J1006 to J21, TP1006 to TP2
Connections:
- net PCIE30_TX0_N: no longer names the net of J21.B15 (PETn0)
- net PCIE30_TX0_P: no longer names the net of J21.B14 (PETp0)
- net PCIE_RX_0+: no longer names the net of J21.A16 (PERp0)
- net PCIE_RX_0-: no longer names the net of J21.A17 (PERn0)
- net REFCLK+: no longer names the net of J21.A13 (REFCLK+)
- net REFCLK-: no longer names the net of J21.A14 (REFCLK-)
