File: PSU.kicad_sch (KiCad schematic)
At the start: 97 parts, among them Q1 2N7002, Q10 AO3407, Q2 2N7002, Q3 NCE30P28Q, Q4 2N7002, Q5 2N7002, Q6 2N7002, Q7 2N7002, Q8 2N7002, Q9 2N7002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

Commit message: before board exclusion
Parts:
- added J9: Barrel_Jack, A_DFRobot:DC_Jack_DC007B_30V_10A, symbol Connector:Barrel_Jack
- added R151: 0, Resistor_SMD:R_2010_5025Metric, symbol Library:R
Connections:
- net GND is gone; now on net QGND: C160.2, C162.1, C163.1, C164.1, C165.1, Q2.2 (S), R87.1, R90.1, U39.3 (A)
- net QGND: now also J9.1
- net SUPPLY_PWR: now also R151.1
- net at C160.1, Q1.1 (G), R90.2: now also R89.1
- new net: J9.2, R151.2
Other:
- moved on the sheet: NT2
