File: PSU.kicad_sch (KiCad schematic)
At the start: 69 parts, among them J6 Conn_01x01_Socket, Q401 2N7002, SW401 SW_Push, SW402 SW_Push, U3 TPPM0110DWPR, U4 TPS548A23VANR, U402 AP7381-33SA-7, U403 AP63200WU

Commit message: added MPN to all parts by hand :'(
Parts:
- C10, C12, C8, C9: footprint Capacitor_SMD:C_1206_3216Metric -> A_DFRobot:C_0805_2012Metric; MPN GRM31CC81E226ME11L -> GRM21BR61E226ME44L
- C2, C3, C4, C5, C6: footprint Capacitor_SMD:C_0805_2012Metric -> A_DFRobot:C_0603; MPN C2012X5R1E106K125AB -> GRM188R61E106KA73D
- C401, C405: value 100n -> u1; MPN 478-KGM05CR71H104KHCT-ND -> C1005X7R1H104K050BE
- C402: MPN 490-5942-1-ND -> C0402C470J5GACTU
- C403, C404: footprint A_HDJ_Library:C_0603_1608Metric -> A_DFRobot:C_0805_2012Metric; Digikey 490-10476-1-ND -> (none); MPN 490-10476-1-ND -> GRM21BR61E226ME44L
- C408: Digikey 445-14428-1-ND -> (none); MPN 445-14428-1-ND -> GRM21BR61E226ME44L
- C414, C415: MPN 490-GRM155R61H105KE05DCT-ND -> C1005X7R1H104K050BE
- C416, C417: Digikey 490-GRM155R61H105KE05DCT-ND -> (none); MPN 490-GRM155R61H105KE05DCT-ND -> GRM155R61H105KE05D
- R18: MPN ERJ-2RKF1003X -> RCS0402100KFKED
- R22: MPN ERJPA2F1002X -> RCS040210K0FKED
- R401: Digikey 311-100KJRCT-ND -> (none); MPN 311-100KJRCT-ND -> RCS0402100KFKED
- R402: Digikey 13-RC0402FR-1319K1LCT-ND -> (none); MPN 13-RC0402FR-1319K1LCT-ND -> CRCW040219K1FKED
- R405: MPN 311-1.0KJRCT-ND -> RCS04021K00JNED
- R406, R407, R408: Digikey 311-1.0KJRCT-ND -> (none); MPN 311-1.0KJRCT-ND -> RCS04021K00JNED
- R409: Digikey 311-10KJRCT-ND -> (none); MPN 311-10KJRCT-ND -> RCS040210K0FKED
- U3: MPN (none) -> TPPM0110DWPR
- U4: MPN (none) -> TPS548A23VANR
Changed lines of the file:
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@@
 			)
 		)
-		(property "MPN" "490-5942-1-ND"
+		(property "MPN" "C0402C470J5GACTU"
 			(at 273.05 190.5 90)
 			(hide yes)
@@
 			)
 		)
-		(property "Digikey" "13-RC0402FR-1319K1LCT-ND"
+		(property "Digikey" ""
 			(at 265.43 198.12 0)
 			(hide yes)
@@
 			)
 		)
-		(property "MPN" "13-RC0402FR-1319K1LCT-ND"
+		(property "MPN" "CRCW040219K1FKED"
 			(at 265.43 198.12 0)
 			(hide yes)
@@
 			)
 		)
-		(property "Digikey" "311-100KJRCT-ND"
+		(property "Digikey" ""
 			(at 265.43 190.5 0)
 			(hide yes)
@@
 			)
 		)
-		(property "MPN" "311-100KJRCT-ND"
+		(property "MPN" "RCS0402100KFKED"
 			(at 265.43 190.5 0)
 			(hide yes)
@@
 			)
 		)
-		(property "MPN" "ERJPA2F1002X"
+		(property "MPN" "RCS040210K0FKED"
 			(at 461.01 222.25 90)
 			(hide yes)
@@
 			)
 		)
-		(property "Digikey" "311-1.0KJRCT-ND"
+		(property "Digikey" ""
 			(at 152.4 233.68 90)
 			(hide yes)
@@
 			)
 		)
-		(property "MPN" "311-1.0KJRCT-ND"
+		(property "MPN" "RCS04021K00JNED"
 			(at 152.4 233.68 90)
 			(hide yes)
@@
 			)
 		)
-		(property "Footprint" "Capacitor_SMD:C_1206_3216Metric"
+		(property "Footprint" "A_DFRobot:C_0805_2012Metric"
 			(at 380.6952 186.69 0)
 			(hide yes)
@@
 			)
 		)
-		(property "MPN" "GRM31CC81E226ME11L"
+		(property "MPN" "GRM21BR61E226ME44L"
 			(at 379.73 182.88 0)
 			(hide yes)
@@
 			)
 		)
-		(property "Footprint" "Capacitor_SMD:C_1206_3216Metric"
+		(property "Footprint" "A_DFRobot:C_0805_2012Metric"
 			(at 364.1852 186.69 0)
 			(hide yes)
@@
 			)
 		)
-		(property "MPN" "GRM31CC81E226ME11L"
+		(property "MPN" "GRM21BR61E226ME44L"
 			(at 363.22 182.88 0)
 			(hide yes)
@@
 			)
 		)
-		(property "Footprint" "Capacitor_SMD:C_0805_2012Metric"
+		(property "Footprint" "A_DFRobot:C_0603"
 			(at 457.5048 74.93 0)
 			(hide yes)
@@
 			)
 		)
-		(property "MPN" "C2012X5R1E106K125AB"
+		(property "MPN" "GRM188R61E106KA73D"
 			(at 458.47 78.74 0)
 			(hide yes)
@@
 			)
 		)
-		(property "Digikey" "490-GRM155R61H105KE05DCT-ND"
+		(property "Digikey" ""
 			(at 180.34 302.26 0)
 			(hide yes)
@@
 			)
 		)
-		(property "MPN" "490-GRM155R61H105KE05DCT-ND"
+		(property "MPN" "GRM155R61H105KE05D"
 			(at 180.34 302.26 0)
 			(hide yes)
@@
 			)
 		)
-		(property "MPN" "490-GRM155R61H105KE05DCT-ND"
+		(property "MPN" "C1005X7R1H104K050BE"
 			(at 170.18 320.04 0)
 			(hide yes)
@@
 			)
 		)
-		(property "Footprint" "Capacitor_SMD:C_0805_2012Metric"
+		(property "Footprint" "A_DFRobot:C_0603"
 			(at 477.8248 74.93 0)
 			(hide yes)
@@
 			)
 		)
-		(property "MPN" "C2012X5R1E106K125AB"
+		(property "MPN" "GRM188R61E106KA73D"
 			(at 478.79 78.74 0)
 			(hide yes)
@@
 			)
 		)
-		(property "Digikey" "311-1.0KJRCT-ND"
-			(at 304.8 254 90)
-			(hide yes)
-			(show_name no)
-			(do_not_autoplace no)
-			(effects
-				(font
-					(size 1.27 1.27)
-				)
-			)
-		)
-		(property "MPN" "311-1.0KJRCT-ND"
+		(property "Digikey" ""
 			(at 304.8 254 90)
 			(hide yes)
@@
 			)
 		)
-		(property "Field11" ""
+		(property "MPN" "RCS04021K00JNED"
 			(at 304.8 254 90)
 			(hide yes)
@@
 			)
 		)
-		(property "Value" "100n"
+		(property "Value" "u1"
 			(at 247.65 182.88 90)
 			(show_name no)
@@
 			)
 		)
-		(property "MPN" "478-KGM05CR71H104KHCT-ND"
+		(property "MPN" "C1005X7R1H104K050BE"
 			(at 248.92 186.69 90)
 			(hide yes)
@@
 			)
 		)
-		(property "Digikey" "311-10KJRCT-ND"
+		(property "Digikey" ""
 			(at 312.42 257.81 0)
 			(hide yes)
@@
 			)
 		)
-		(property "MPN" "311-10KJRCT-ND"
+		(property "MPN" "RCS040210K0FKED"
 			(at 312.42 257.81 0)
 			(hide yes)
@@
 			)
 		)
-		(property "Footprint" "A_HDJ_Library:C_0603_1608Metric"
+		(property "Footprint" "A_DFRobot:C_0805_2012Metric"
 			(at 284.7848 190.5 0)
 			(hide yes)
@@
 			)
 		)
-		(property "Digikey" "490-10476-1-ND"
+		(property "Digikey" ""
 			(at 285.75 194.31 90)
 			(hide yes)
@@
 			)
 		)
-		(property "MPN" "490-10476-1-ND"
+		(property "MPN" "GRM21BR61E226ME44L"
 			(at 285.75 194.31 90)
 			(hide yes)
@@
 			)
 		)
-		(property "Footprint" "Capacitor_SMD:C_0805_2012Metric"
+		(property "Footprint" "A_DFRobot:C_0603"
 			(at 467.6648 74.93 0)
 			(hide yes)
@@
 			)
 		)
-		(property "MPN" "C2012X5R1E106K125AB"
+		(property "MPN" "GRM188R61E106KA73D"
 			(at 468.63 78.74 0)
 			(hide yes)
@@
 			)
 		)
-		(property "Description" "ERJ-2RKF1003X"
+		(property "Description" ""
 			(at 351.79 218.44 0)
 			(hide yes)
@@
 			)
 		)
-		(property "MPN" "ERJ-2RKF1003X"
+		(property "MPN" "RCS0402100KFKED"
 			(at 351.79 218.44 0)
 			(hide yes)
@@
 			)
 		)
-		(property "Footprint" "Capacitor_SMD:C_0805_2012Metric"
+		(property "Footprint" "A_DFRobot:C_0603"
 			(at 438.4548 74.93 0)
 			(hide yes)
@@
 			)
 		)
-		(property "MPN" "C2012X5R1E106K125AB"
+		(property "MPN" "GRM188R61E106KA73D"
 			(at 439.42 78.74 0)
 			(hide yes)
@@
 			)
 		)
+		(property "MPN" "TPPM0110DWPR"
+			(at 196.85 298.45 0)
+			(hide yes)
+			(show_name no)
+			(do_not_autoplace no)
+			(effects
+				(font
+					(size 1.27 1.27)
+				)
+			)
+		)
 		(pin "20"
 		)
@@
 			)
 		)
-		(property "Footprint" "A_HDJ_Library:C_0603_1608Metric"
+		(property "Footprint" "A_DFRobot:C_0805_2012Metric"
 			(at 279.7048 190.5 0)
 			(hide yes)
@@
 			)
 		)
-		(property "Digikey" "490-10476-1-ND"
+		(property "Digikey" ""
 			(at 280.67 194.31 90)
 			(hide yes)
@@
 			)
 		)
-		(property "MPN" "490-10476-1-ND"
+		(property "MPN" "GRM21BR61E226ME44L"
 			(at 280.67 194.31 90)
 			(hide yes)
@@
 			)
 		)
-		(property "Footprint" "Capacitor_SMD:C_1206_3216Metric"
+		(property "Footprint" "A_DFRobot:C_0805_2012Metric"
 			(at 380.6952 167.64 0)
 			(hide yes)
@@
 			)
 		)
-		(property "MPN" "GRM31CC81E226ME11L"
+		(property "MPN" "GRM21BR61E226ME44L"
 			(at 379.73 163.83 0)
 			(hide yes)
@@
 			)
 		)
-		(property "MPN" "490-GRM155R61H105KE05DCT-ND"
+		(property "MPN" "C1005X7R1H104K050BE"
 			(at 170.18 302.26 0)
 			(hide yes)
@@
 			)
 		)
-		(property "Footprint" "Capacitor_SMD:C_0805_2012Metric"
+		(property "Footprint" "A_DFRobot:C_0603"
 			(at 447.3448 74.93 0)
 			(hide yes)
@@
 			)
 		)
-		(property "MPN" "C2012X5R1E106K125AB"
+		(property "MPN" "GRM188R61E106KA73D"
 			(at 448.31 78.74 0)
 			(hide yes)
@@
 			)
 		)
-		(property "MPN" "311-1.0KJRCT-ND"
+		(property "MPN" "RCS04021K00JNED"
 			(at 114.3 233.68 90)
 			(hide yes)
@@
 			)
 		)
-		(property "Value" "100n"
+		(property "Value" "u1"
 			(at 292.1 200.66 90)
 			(show_name no)
@@
 			)
 		)
-		(property "MPN" "478-KGM05CR71H104KHCT-ND"
+		(property "MPN" "C1005X7R1H104K050BE"
 			(at 290.83 194.31 90)
 			(hide yes)
@@
 			)
 		)
-		(property "Footprint" "Capacitor_SMD:C_1206_3216Metric"
+		(property "Footprint" "A_DFRobot:C_0805_2012Metric"
 			(at 362.9152 167.64 0)
 			(hide yes)
@@
 			)
 		)
-		(property "MPN" "GRM31CC81E226ME11L"
+		(property "MPN" "GRM21BR61E226ME44L"
 			(at 361.95 163.83 0)
 			(hide yes)
@@
 			)
 		)
-		(property "Digikey" "490-GRM155R61H105KE05DCT-ND"
+		(property "Digikey" ""
 			(at 180.34 320.04 0)
 			(hide yes)
@@
 			)
 		)
-		(property "MPN" "490-GRM155R61H105KE05DCT-ND"
+		(property "MPN" "GRM155R61H105KE05D"
 			(at 180.34 320.04 0)
 			(hide yes)
@@
 			)
 		)
+		(property "MPN" "TPS548A23VANR"
+			(at 412.75 196.85 0)
+			(hide yes)
+			(show_name no)
+			(do_not_autoplace no)
+			(effects
+				(font
+					(size 1.27 1.27)
+				)
+			)
+		)
 		(pin "6"
 		)
@@
 			)
 		)
-		(property "Digikey" "445-14428-1-ND"
+		(property "Digikey" ""
 			(at 191.77 195.58 90)
 			(hide yes)
@@
 			)
 		)
-		(property "MPN" "445-14428-1-ND"
+		(property "MPN" "GRM21BR61E226ME44L"
 			(at 191.77 195.58 90)
 			(hide yes)
@@
 			)
 		)
-		(property "Digikey" "311-1.0KJRCT-ND"
+		(property "Digikey" ""
 			(at 323.85 237.49 0)
 			(hide yes)
@@
 			)
 		)
-		(property "MPN" "311-1.0KJRCT-ND"
+		(property "MPN" "RCS04021K00JNED"
 			(at 323.85 237.49 0)
 			(hide yes)

Commit message: Prototype
Parts:
- added H14, H15: MountingHole_Pad, Connector:Banana_Jack_1Pin, symbol Mechanical:MountingHole_Pad
- C416, C417: footprint A_HDJ_Library:C_0402_1005Metric -> A_DFRobot:C_0603; MPN GRM155R61H105KE05D -> GZ1608D601TF
Connections:
- net +12V: now also H15.1
- net GND: now also H14.1
