File: USBPD.kicad_sch (KiCad schematic)
At the start: 92 parts, among them J21 USB_C_Receptacle_USB2.0, J3 TS NORMAL, J33 Conn_02x02_Odd_Even, J4 EXTERNAL THERMISTOR GND, J5 2S 1.5MHz 2A ICHG, J6 3S 1.5MHz 1A ICHG, J8 4S 1.5MHz 1A ICHG, U1 CAT24C512WI-GT3, U2 TPS25750DRJKR, U3 BQ25792RQMR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

Commit message: before board exclusion
Parts:
- NT1: footprint NetTie:NetTie-3_SMD_Pad2.0mm -> NetTie:NetTie-2_SMD_Pad0.5mm
Connections:
- net GND is gone; now on net PGND: C15.2, C20.1, C23.1, C27.1, C30.1, C31.1
Other:
- moved on the sheet: R24
