File: USBPD.kicad_sch (KiCad schematic)
At the start: 93 parts, among them J1001 USB_C_Receptacle, J16 Conn_02x05_Odd_Even, J17 TS NORMAL, J18 EXTERNAL THERMISTOR GND, J22 2S 1.5MHz 2A ICHG, J23 3S 1.5MHz 1A ICHG, J24 4S 1.5MHz 1A ICHG, J26 BATTERY GND, U1004 CAT24C512WI-GT3, U1006 TVS2200DRVR, U2 TPS25750DRJKR, U22 TLV75533PDBVR, U23 TPS54531DDAR, U3 BQ25792RQMR

Commit message: commit before removing duplicated glasgow
Parts:
- removed J16: Conn_02x05_Odd_Even, symbol Connector_Generic:Conn_02x05_Odd_Even
- removed J26: BATTERY GND, symbol Connector_Generic:Conn_01x02
- added J33: Conn_02x02_Odd_Even, Connector_PinHeader_1.00mm:PinHeader_2x02_P1.00mm_Vertical_SMD, symbol Connector_Generic:Conn_02x02_Odd_Even
- J3: renamed from J17; footprint (none) -> Connector_PinHeader_1.00mm:PinHeader_1x02_P1.00mm_Vertical
- J4: renamed from J18; footprint (none) -> PowerShit:CONN_SD-39357-001_02P_MOL
- J5: renamed from J22; footprint (none) -> Connector_PinHeader_1.00mm:PinHeader_1x02_P1.00mm_Vertical
- J6: renamed from J23; footprint (none) -> Connector_PinHeader_1.00mm:PinHeader_1x02_P1.00mm_Vertical
- J8: renamed from J24; footprint (none) -> Connector_PinHeader_1.00mm:PinHeader_1x02_P1.00mm_Vertical
- U3: footprint RQM0029A-MFG -> PowerShit:RQM0029A-MFG
- renumbered C9 to C1, C1032 to C10, C1024 to C11, C13 to C12, C18 to C13, C1026 to C14, C1030 to C15, C59 to C16, C6 to C17, C19 to C18, C20 to C19, C1027 to C2, C51 to C20, C7 to C21, C1037 to C22, C52 to C23, C8 to C24, C1035 to C25, C4 to C26, C1031 to C27, C5 to C28, C1036 to C29, C10 to C3, C1033 to C30, C1034 to C31, C60 to C32, C62 to C33, C63 to C34, C64 to C35, C1038 to C36, C65 to C37, C68 to C38, C1042 to C39, C1028 to C4, C1043 to C40, C1044 to C41, C66 to C42, C1045 to C43, C67 to C44, C1046 to C45, C69 to C46, C70 to C47, C1041 to C48, C11 to C5, C1029 to C6, C1025 to C7, C12 to C8, C1 to C9, D14 to D1, D15 to D2, FB1001 to FB1, J1001 to J9, R4 to R10, R33 to R11, R1027 to R12, R1026 to R13, R34 to R14, R36 to R15, R35 to R16, R38 to R17, R37 to R18, R43 to R19, R39 to R20, R40 to R21, R41 to R22, R42 to R23, R44 to R24, R45 to R25, R46 to R26, R47 to R27, R48 to R28, R49 to R29, R32 to R5, R1029 to R6, R3 to R7, R1028 to R8, R31 to R9, U1004 to U1, U22 to U4, U23 to U5, U1006 to U6
Connections:
- net VBUS_POWER is gone; now on net VBUS_PD: FB1.2
- net GNDA: now also J33.3 (Pin_3)
- net at R11.1: now also J33.4 (Pin_4)
- net BAT renamed BATT_SUPPLY
- net I2C0_SCL renamed PD_I2C0_SCL
- net I2C0_SDA renamed PD_I2C0_SDA
- net I2C1_SCL renamed PD_I2C1_SCL
- net PD_I2C1_SCL: now also J33.2 (Pin_2)
- net I2C1_SDA renamed PD_I2C1_SDA
- net PD_I2C1_SDA: now also J33.1 (Pin_1)
- net VBUS renamed VBUS_PD

Commit message: is this a differential pair?
Parts:
- removed J9: USB_C_Receptacle, Glasgow:USB_C_Receptacle_HRO_TYPE-C-31-M-12, symbol Connector:USB_C_Receptacle
- added J21: USB_C_Receptacle_USB2.0, Glasgow:USB_C_Receptacle_HRO_TYPE-C-31-M-12, symbol glasgow:USB_C_Receptacle_USB2.0
- C1, C13, C2, C25, C29, C3, C32, C36, C37, C39, C4, C42, C44, C5, C6, C8, R23: DF_Comment (none) -> 贴片电容0603-22uF-10V-X5R(0603); SCH_Show_Footprint (none) -> C603
- C10, C11, C12, C14, C15, C16, C18, C19, C22, C24, C38, C40, C41, C43, C45, C7, C9: DF_Comment (none) -> 贴片电容0402-10UF-10V-X5R_GRM155R61A106ME44D; SCH_Show_Footprint (none) -> C0402
- C46: footprint CAPMP3.7X2.8_2N_KEM -> PowerShit:CAPMP3.7X2.8_2N_KEM
- FB1: Buy_Link (none) -> https://item.szlcsc.com/947787.html; DF_Comment (none) -> 0805贴片自恢复保险丝2A/6V-BSMD0805L-200; SCH_Show_Footprint (none) -> R0805
- R11, R17, R18, R19, R24, R25, R26, R27, R28, R29: Buy_Link (none) -> https://item.szlcsc.com/8530937.html; DF_Comment (none) -> 0603贴片自恢复保险丝0.05A/6V-0603L005/6AR; SCH_Show_Footprint (none) -> R0805
- R14, R15, R16, R20: DF_Comment (none) -> 贴片电阻0402-10K-1%
- U1: footprint SOIC8_ONS -> PowerShit:SOIC8_ONS
- U2: footprint RJK0038B-C01-MFG -> PowerShit:RJK0038B-C01-MFG
- U4: footprint DBV0005A_N -> PowerShit:DBV0005A_N
- U5: footprint DDA8_3P1X2P4_TEX -> PowerShit:DDA8_3P1X2P4_TEX
Connections:
- net C_CC1: now also J21.A5 (CC1)
- net C_CC2: now also J21.B5 (CC2)
- net C_USB_N: now also J21.A7 (D-), J21.B7 (D-)
- net C_USB_P: now also J21.A6 (D+), J21.B6 (D+)
- net PGND: now also J21.A1 (GND), J21.A12 (GND), J21.B1 (GND), J21.B12 (GND), J21.S1 (SHIELD)
- net at C39.2, C40.2, C41.2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: now also J21.A4 (VBUS), J21.A9 (VBUS), J21.B4 (VBUS), J21.B9 (VBUS)
- no-connect marks 28 -> 18

Commit message: went back to the drawing board
Parts:
- removed C1, C2, C25, C29, C3, C32, C36, C4, C5, C6, C8: 10uF, A_HDJ_Library:C_0603_1608Metric, symbol Device:C
- removed C10, C12, C15, C22, C24, C38: 0.1uF, A_HDJ_Library:C_0402_1005Metric, symbol Device:C
- removed C11, C7, C9: 10V 10uF, A_HDJ_Library:C_0402_1005Metric, symbol Device:C
- removed C13, C39: 4.7uF, A_HDJ_Library:C_0603_1608Metric, symbol Device:C
- removed C14: 0.1uF 35v, A_HDJ_Library:C_0402_1005Metric, symbol Device:C
- removed C16: 50V 1000pF, A_HDJ_Library:C_0402_1005Metric, symbol Device:C
- removed C17, C21: 22uF, PowerShit:CAP_2012_TDK, symbol Device:C
- removed C18, C19: 0.047uF, A_HDJ_Library:C_0402_1005Metric, symbol Device:C
- removed C20: 10uF, Capacitor_SMD:C_0805_2012Metric, symbol Device:C
- removed C23, C27, C30, C31: 10uF 25V, Capacitor_SMD:C_0805_2012Metric, symbol Device:C
- removed C26, C28: 330pF, Capacitor_SMD:C_0201_0603Metric, symbol Device:C
- removed C33, C34: 50V 4.7uF, Capacitor_SMD:C_1210_3225Metric, symbol Device:C
- removed C35: 10nF 50V, Capacitor_SMD:C_0805_2012Metric, symbol Device:C
- removed C37: 10nF 100V, A_HDJ_Library:C_0603_1608Metric, symbol Device:C
- removed C40, C41, C43, C45: .01 uF, A_HDJ_Library:C_0402_1005Metric, symbol Device:C
- removed C42: 2.2nF 50V, A_HDJ_Library:C_0603_1608Metric, symbol Device:C
- removed C44: 50V 22pF, A_HDJ_Library:C_0603_1608Metric, symbol Device:C
- removed C46: T520B107M006ATE015, PowerShit:CAPMP3.7X2.8_2N_KEM, symbol T520B107M006ATE015:T520B107M006ATE015
- removed C47, C48: 10V 47uF, Capacitor_SMD:C_1210_3225Metric, symbol Device:C
- removed D1: LED, PowerShit:LED_LTST-C190CKT_LTO, symbol Device:LED
- removed D2: CDBC540-G, PowerShit:CDBC-G, symbol Device:D_Schottky
- removed FB1: FerriteBead, A_HDJ_Library:R_0805_2012Metric, symbol Device:FerriteBead
- removed J21: USB_C_Receptacle_USB2.0, Glasgow:USB_C_Receptacle_HRO_TYPE-C-31-M-12, symbol glasgow:USB_C_Receptacle_USB2.0
- removed J3: TS NORMAL, Connector_PinHeader_1.00mm:PinHeader_1x02_P1.00mm_Vertical, symbol Connector_Generic:Conn_01x02
- removed J33: Conn_02x02_Odd_Even, Connector_PinHeader_1.00mm:PinHeader_2x02_P1.00mm_Vertical_SMD, symbol Connector_Generic:Conn_02x02_Odd_Even
- removed J4: EXTERNAL THERMISTOR GND, PowerShit:CONN_SD-39357-001_02P_MOL, symbol Connector_Generic:Conn_01x02
- removed J5: 2S 1.5MHz 2A ICHG, Connector_PinHeader_1.00mm:PinHeader_1x02_P1.00mm_Vertical, symbol Connector_Generic:Conn_01x02
- removed J6: 3S 1.5MHz 1A ICHG, Connector_PinHeader_1.00mm:PinHeader_1x02_P1.00mm_Vertical, symbol Connector_Generic:Conn_01x02
- removed J8: 4S 1.5MHz 1A ICHG, Connector_PinHeader_1.00mm:PinHeader_1x02_P1.00mm_Vertical, symbol Connector_Generic:Conn_01x02
- removed L1: 1uH, PowerShit:IND_IHLP-2020BZ_VIS, symbol Device:L_Iron
- removed L2: 4.7uH, PowerShit:IND_1040-WE-LHMI_WRE, symbol Device:L_Iron
- removed NT1: NetTie_2, NetTie:NetTie-3_SMD_Pad2.0mm, symbol Device:NetTie_2
- removed R10, R7: 2.20K/1%, Resistor_SMD:R_0201_0603Metric, symbol Device:R
- removed R11: 10.0, A_HDJ_Library:R_0603_1608Metric, symbol Library:R
- removed R12, R13, R6, R8: 10K, Resistor_SMD:R_0201_0603Metric, symbol Library:R
- removed R14: 30.1k, A_HDJ_Library:R_0402_1005Metric, symbol Library:R
- removed R15: 5.23k, A_HDJ_Library:R_0402_1005Metric, symbol Library:R
- removed R16: 10k, A_HDJ_Library:R_0402_1005Metric, symbol Library:R
- removed R17: 100k, A_HDJ_Library:R_0603_1608Metric, symbol Library:R
- removed R18: 137k, A_HDJ_Library:R_0603_1608Metric, symbol Library:R
- removed R19: 100 Ohm, A_HDJ_Library:R_0603_1608Metric, symbol Library:R
- removed R20: 2.21K, A_HDJ_Library:R_0402_1005Metric, symbol Library:R
- removed R21: 6.04k, Resistor_SMD:R_0201_0603Metric, symbol Library:R
- removed R22: 10.5k, Resistor_SMD:R_0201_0603Metric, symbol Library:R
- removed R23: 17.4k, A_HDJ_Library:C_0603_1608Metric, symbol Library:R
- removed R24: 665k, A_HDJ_Library:R_0603_1608Metric, symbol Library:R
- removed R25: 130k, A_HDJ_Library:R_0603_1608Metric, symbol Library:R
- removed R26: 37.4k, A_HDJ_Library:R_0603_1608Metric, symbol Library:R
- removed R27: 51.1, A_HDJ_Library:R_0603_1608Metric, symbol Library:R
- removed R28: 10.2k, A_HDJ_Library:R_0603_1608Metric, symbol Library:R
- removed R29: 1.96k, A_HDJ_Library:R_0603_1608Metric, symbol Library:R
- removed R5, R9: 2.20k, Resistor_SMD:R_0201_0603Metric, symbol Library:R
- removed U1: CAT24C512WI-GT3, PowerShit:SOIC8_ONS, symbol 2026-03-23_00-21-58:CAT24C512WI-GT3
- removed U2: TPS25750DRJKR, PowerShit:RJK0038B-C01-MFG, symbol TPS25750DRJKR _2026-03-20_15-46-48:TPS25750DRJKR
- removed U3: BQ25792RQMR, PowerShit:RQM0029A-MFG, symbol 2026-03-20_06-56-57:BQ25792RQMR
- removed U4: TLV75533PDBVR, PowerShit:DBV0005A_N, symbol TLV5533PDBVR:TLV75533PDBVR
- removed U5: TPS54531DDAR, PowerShit:DDA8_3P1X2P4_TEX, symbol 2026-03-20_06-57-59:TPS54531DDAR
- removed U6: TVS2200DRVR, PowerShit:SON65P200X200X80-7N, symbol TVS2200DRVR:TVS2200DRVR
- added C51: 0.1uF, A_HDJ_Library:C_0402_1005Metric, symbol Device:C
- added C52: 10uF, Capacitor_SMD:C_0805_2012Metric, symbol Device:C
- added C53, C54, C55, C56: 10uF 25V, Capacitor_SMD:C_0805_2012Metric, symbol Device:C
Connections:
- net GND: now also C51.2, C52.1, C53.1, C54.1, C55.1, C56.1
- new net +12V: C51.1, C52.2, C53.2, C54.2, C55.2, C56.2
- no-connect marks 18 -> 0
