File: extendo.kicad_sch (KiCad schematic)
At the start: 2 parts, among them J7 Barrel_Jack, P1 1775862-2

Commit message: is this a differential pair?
Parts:
- J7: Buy_Link (none) -> https://item.szlcsc.com/19360929.html; DF_Comment (none) -> DC2.5电源母座_12V/10A_XDJK-060B-055
Changed lines of the file:
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@@
+			)
+		)
+		(property "Buy_Link" "https://item.szlcsc.com/19360929.html"
+			(at 205.74 86.36 0)
+			(effects
+				(font
+					(size 1.27 1.27)
+				)
+				(hide yes)
+			)
+		)
+		(property "DF_Comment" "DC2.5电源母座_12V/10A_XDJK-060B-055"
+			(at 205.74 86.36 0)
+			(effects
+				(font
+					(size 1.27 1.27)
+				)
+				(hide yes)
+			)
+		)
+		(property "Field-1" ""
+			(at 205.74 86.36 0)
+			(effects
+				(font
+					(size 1.27 1.27)
+				)
+				(hide yes)
+			)
+		)
+		(property "SCH_Show_Footprint" ""
+			(at 205.74 86.36 0)
+			(effects
+				(font
+					(size 1.27 1.27)
+				)
+				(hide yes)
+			)
+		)
+		(property "无标题字段" ""
+			(at 205.74 86.36 0)
+			(effects
+				(font
+					(size 1.27 1.27)
+				)
+				(hide yes)
 			)
 		)

Commit message: before board exclusion
Parts:
- J7: now not fitted
Changed lines of the file:
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@@
 		(exclude_from_sim no)
 		(in_bom yes)
-		(on_board yes)
-		(dnp no)
+		(on_board no)
+		(dnp yes)
 		(fields_autoplaced yes)
 		(property "Reference" "J7"
