File: extendo.kicad_sch (KiCad schematic)
At the start: 2 parts, among them J7 Barrel_Jack, P1 1775862-2

Commit message: went back to the drawing board
Parts:
- removed J7: Barrel_Jack, A_DFRobot:DC_Jack_DC007B_30V_10A, symbol Connector:Barrel_Jack
Connections:
- net GND: now also P1.17 (UIM_C8/RES), P1.18 (GND4), P1.19 (UIM_C4/RES), P1.20 (~{W_DISABLE}/RES), P1.21 (GND5), P1.22 (~{PERST}/RES), P1.23 (PERN0/+B), P1.24 (+3.3VAUX/+3.3V2), P1.25 (PERP0/-B), P1.26 (GND6), P1.27 (GND7), P1.28 (+1.5V1), P1.29 (GND9)
- net +12V: now reaches P1.38 (USB_D+/RES)
- net +12V: now also P1.39 (+3.3VAUX/+3.3V3), P1.40 (GND10), P1.41 (+3.3VAUX/+3.3V4), P1.42 (~{LED_WWAN}/RES), P1.43 (GND/NC), P1.44 (~{LED_WLAN}/RES), P1.45 (RES/VENDOR1), P1.46 (~{LED_WPAN}/RES), P1.47 (RES/VENDOR2), P1.48 (+1.5V2), P1.49 (RES/DA/DSS), P1.50 (GND12), P1.51 (RES/DETECT), P1.52 (+3.3VAUX/+3.3V5)
- removed net PD_GND: P1.15 (GND3), P1.18 (GND4), P1.21 (GND5), P1.26 (GND6), P1.27 (GND7), P1.29 (GND9), P1.34 (GND8), P1.35 (GND11), P1.37 (GND13), P1.4 (GND2), P1.40 (GND10), P1.43 (GND/NC), P1.50 (GND12), P1.9 (GND1)
- removed net PD_SUPPLY: P1.2 (3.3VAUX/+3.3V1), P1.24 (+3.3VAUX/+3.3V2), P1.28 (+1.5V1), P1.48 (+1.5V2), P1.52 (+3.3VAUX/+3.3V5), P1.6 (1.5V/+1.5V)

Commit message: rpi edgeboard
Connections:
- net GPIO_5: now reaches P1.10 (UIM_DATA/RES)
- net GPIO_6: now reaches P1.12 (UIM_CLK/RES)
- net GPIO_7: now reaches P1.14 (UIM_RESET/RES)
- net GPIO_8: now reaches P1.16 (UIM_VPP/RES)
- net GPIO_1: now reaches P1.2 (3.3VAUX/+3.3V1)
- net GPIO_2: now reaches P1.4 (GND2)
- net GPIO_3: now reaches P1.6 (1.5V/+1.5V)
- net GPIO_4: now reaches P1.8 (UIM_PWR/RES)
Changed lines of the file:
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@@
+		)
+	)
+	(hierarchical_label "GPIO_1"
+		(shape input)
+		(at 107.95 69.85 0)
+		(effects
+			(font
+				(size 1.27 1.27)
+			)
+			(justify left)
+		)
+	)
+	(hierarchical_label "GPIO_3"
+		(shape input)
+		(at 107.95 74.93 0)
+		(effects
+			(font
+				(size 1.27 1.27)
+			)
+			(justify left)
+		)
+	)
+	(hierarchical_label "GPIO_2"
+		(shape input)
+		(at 107.95 72.39 0)
+		(effects
+			(font
+				(size 1.27 1.27)
+			)
+			(justify left)
+		)
+	)
+	(hierarchical_label "GPIO_8"
+		(shape input)
+		(at 107.95 87.63 0)
+		(effects
+			(font
+				(size 1.27 1.27)
+			)
+			(justify left)
+		)
+	)
+	(hierarchical_label "GPIO_4"
+		(shape input)
+		(at 107.95 77.47 0)
+		(effects
+			(font
+				(size 1.27 1.27)
+			)
+			(justify left)
 		)
 	)
@@
 		(effects
 			(font
+				(size 1.27 1.27)
+			)
+			(justify left)
+		)
+	)
+	(hierarchical_label "GPIO_6"
+		(shape input)
+		(at 107.95 82.55 0)
+		(effects
+			(font
+				(size 1.27 1.27)
+			)
+			(justify left)
+		)
+	)
+	(hierarchical_label "GPIO_7"
+		(shape input)
+		(at 107.95 85.09 0)
+		(effects
+			(font
+				(size 1.27 1.27)
+			)
+			(justify left)
+		)
+	)
+	(hierarchical_label "GPIO_5"
+		(shape input)
+		(at 107.95 80.01 0)
+		(effects
+			(font

Commit message: V4 done ???
Connections:
- net GPIO_1: now also P1.4 (GND2); no longer P1.2 (3.3VAUX/+3.3V1)
- net GPIO_2: now also P1.6 (1.5V/+1.5V); no longer P1.4 (GND2)
- net GPIO_3: now also P1.8 (UIM_PWR/RES); no longer P1.6 (1.5V/+1.5V)
- net GPIO_4: now also P1.10 (UIM_DATA/RES); no longer P1.8 (UIM_PWR/RES)
- net GPIO_5: now also P1.12 (UIM_CLK/RES); no longer P1.10 (UIM_DATA/RES)
- net GPIO_6: now also P1.14 (UIM_RESET/RES); no longer P1.12 (UIM_CLK/RES)
- net GPIO_7: now also P1.16 (UIM_VPP/RES); no longer P1.14 (UIM_RESET/RES)
- net GPIO_8: now also P1.2 (3.3VAUX/+3.3V1); no longer P1.16 (UIM_VPP/RES)
Changed lines of the file:
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@@
 	(hierarchical_label "GPIO_1"
+		(shape input)
+		(at 107.95 72.39 0)
+		(effects
+			(font
+				(size 1.27 1.27)
+			)
+			(justify left)
+		)
+	)
+	(hierarchical_label "GPIO_3"
+		(shape input)
+		(at 107.95 77.47 0)
+		(effects
+			(font
+				(size 1.27 1.27)
+			)
+			(justify left)
+		)
+	)
+	(hierarchical_label "GPIO_2"
+		(shape input)
+		(at 107.95 74.93 0)
+		(effects
+			(font
+				(size 1.27 1.27)
+			)
+			(justify left)
+		)
+	)
+	(hierarchical_label "GPIO_8"
 		(shape input)
 		(at 107.95 69.85 0)
@@
 		)
 	)
-	(hierarchical_label "GPIO_3"
-		(shape input)
-		(at 107.95 74.93 0)
-		(effects
-			(font
-				(size 1.27 1.27)
-			)
-			(justify left)
-		)
-	)
-	(hierarchical_label "GPIO_2"
-		(shape input)
-		(at 107.95 72.39 0)
-		(effects
-			(font
-				(size 1.27 1.27)
-			)
-			(justify left)
-		)
-	)
-	(hierarchical_label "GPIO_8"
-		(shape input)
-		(at 107.95 87.63 0)
-		(effects
-			(font
-				(size 1.27 1.27)
-			)
-			(justify left)
-		)
-	)
 	(hierarchical_label "GPIO_4"
 		(shape input)
-		(at 107.95 77.47 0)
+		(at 107.95 80.01 0)
 		(effects
 			(font
@@
 	(hierarchical_label "GPIO_6"
 		(shape input)
-		(at 107.95 82.55 0)
+		(at 107.95 85.09 0)
 		(effects
 			(font
@@
 	(hierarchical_label "GPIO_7"
 		(shape input)
-		(at 107.95 85.09 0)
+		(at 107.95 87.63 0)
 		(effects
 			(font
@@
 	(hierarchical_label "GPIO_5"
 		(shape input)
-		(at 107.95 80.01 0)
+		(at 107.95 82.55 0)
 		(effects
 			(font

Commit message: more fixes, tweaks, pretty
Connections:
- net SMB_DATA: now reaches P1.1 (~{WAKE}/RES)
- net SMB_CLK: now reaches P1.3 (COEX1/RES)
- net SMB_ALERT: now reaches P1.5 (COEX2/RES)
Changed lines of the file:
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@@
+		)
+	)
+	(hierarchical_label "SMB_CLK"
+		(shape input)
+		(at 52.07 72.39 180)
+		(effects
+			(font
+				(size 1.27 1.27)
+			)
+			(justify right)
 		)
 	)
@@
 		)
 	)
+	(hierarchical_label "SMB_DATA"
+		(shape bidirectional)
+		(at 52.07 69.85 180)
+		(effects
+			(font
+				(size 1.27 1.27)
+			)
+			(justify right)
+		)
+	)
+	(hierarchical_label "SMB_ALERT"
+		(shape input)
+		(at 52.07 74.93 180)
+		(effects
+			(font
+				(size 1.27 1.27)
+			)
+			(justify right)
+		)
+	)

Commit message: added MPN to all parts by hand :'(
Parts:
- P1: now left out of the parts list
Changed lines of the file:
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@@
 		(body_style 1)
 		(exclude_from_sim no)
-		(in_bom yes)
+		(in_bom no)
 		(on_board yes)
 		(in_pos_files yes)
