File: USB_2_3.kicad_sch (KiCad schematic)
At the start: 0 parts

Commit message: finished schematic draft and started placing components
Parts:
- added C1063, C1064, C1065, C1066: 100nF/16V, A_HDJ_Library:C_0402_1005Metric, symbol Device:C
- added C1067, C1068, C1069: 22uF/10V, A_HDJ_Library:C_0603_1608Metric, symbol Device:C
- added D1010, D1011, D1012, D1013: 0402ESDA-05N, A_HDJ_Library:D_0402_1005Metric, symbol Diode:ESD9B5.0ST5G
- added F2, F3: 6V/1A, A_HDJ_Library:Fuse_0805_2012Metric, symbol Device:Fuse
- added F4, F5: 6V/2A, Fuse:Fuse_0805_2012Metric, symbol Device:Fuse
- added J1003: USB3_A_Stacked, A_HDJ_Library:USB3_A_Molex_48406-0001_Horizontal_Stacked, symbol Connector:USB3_A_Stacked
- added U1008, U1009, U1010: ULC0524P, A_HDJ_Library:Diodes_UDFN-10_1.0x2.5mm_P0.5mm, symbol Power_Protection:D3V3XA4B10LP
Connections:
- new net: F4.2, J1003.1 (VBUS1)
- new net: F5.2, J1003.10 (VBUS2)
- new net +5V: C1067.2, C1068.2, C1069.2, F2.1, F3.1, F4.1, F5.1
- new net CON_USB3_SSTX_N: C1063.2, J1003.8 (SSTX1-), U1008.4, U1008.7 (NC)
- new net CON_USB3_SSTX_P: C1064.2, J1003.9 (SSTX1+), U1008.5, U1008.6 (NC)
- new net CON_USB4_SSTX_N: C1065.2, J1003.17 (SSTX2-), U1008.1, U1008.10 (NC)
- new net CON_USB4_SSTX_P: C1066.2, J1003.18 (SSTX2+), U1008.2, U1008.9 (NC)
- new net GND: C1067.1, C1068.1, C1069.1, D1010.1 (A1), D1011.1 (A1), D1012.1 (A1), D1013.1 (A1), J1003.13 (GND2), J1003.16 (DRAIN2), J1003.19 (SHIELD), J1003.19 (SHIELD), J1003.4 (GND1), J1003.7 (DRAIN1), U1008.3 (VSS), U1008.8 (VSS), U1009.3 (VSS), U1009.8 (VSS), U1010.3 (VSS), U1010.8 (VSS)
- new net USB3_SSRX_N: J1003.5 (SSRX1-), U1010.4, U1010.7 (NC)
- new net USB3_SSRX_P: J1003.6 (SSRX1+), U1010.5, U1010.6 (NC)
- new net USB3_SSTX_N: C1063.1
- new net USB3_SSTX_P: C1064.1
- new net USB4_SSRX_N: J1003.14 (SSRX2-), U1010.1, U1010.10 (NC)
- new net USB4_SSRX_P: J1003.15 (SSRX2+), U1010.2, U1010.9 (NC)
- new net USB4_SSTX_N: C1065.1
- new net USB4_SSTX_P: C1066.1
- new net USB_2_P1+: D1010.2 (A2), J1003.12 (D2+)
- new net USB_2_P1-: D1011.2 (A2), J1003.11 (D2-)
- new net USB_2_P2+: D1012.2 (A2), J1003.3 (D1+)
- new net USB_2_P2-: D1013.2 (A2), J1003.2 (D1-)
- new net USB_2_P3+: U1009.4, U1009.7 (NC)
- new net USB_2_P3-: U1009.5, U1009.6 (NC)
- new net USB_2_P5+: U1009.1, U1009.10 (NC)
- new net USB_2_P5-: U1009.2, U1009.9 (NC)
- new net vbus1_glas: F2.2
- new net vbus2_glas: F3.2

Commit message: commit before removing duplicated glasgow
Parts:
- renumbered C1063 to C81, C1064 to C82, C1065 to C83, C1066 to C84, C1067 to C85, C1068 to C86, C1069 to C87, D1010 to D3, D1011 to D4, D1012 to D5, D1013 to D6, F5 to F1, F4 to F2, F2 to F3, F3 to F4, J1003 to J23, U1008 to U15, U1009 to U16, U1010 to U17
Connections:
- net USB_2_P3+ renamed CON_USB2_D_P
- net USB_2_P3- renamed CON_USB2_D_N

Commit message: REV 0
Changed lines of the file:
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@@
-	(wire
-		(pts
-			(xy 104.1687 39.37) (xy 243.84 39.37)
-		)
-		(stroke
-			(width 0)
-			(type default)
-		)
-	)
 	(wire
 		(pts
@@
 		)
 		(stroke
-			(width 0)
-			(type default)
-		)
-	)
-	(wire
-		(pts
-			(xy 104.1687 41.91) (xy 243.84 41.91)
-		)
-		(stroke
