File: USB_2_3.kicad_sch (KiCad schematic)
At the start: 89 parts, among them J501 USB_C_Receptacle, J502 USB_C_Receptacle, J7 USB3_A, J8 Conn_01x02_Socket, U15 ULC0524P, U16 ULC0524P, U17 ULC0524P, U501 ULC0524P, U502 ULC0524P, U503 ULC0524P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

Commit message: add points to program eeprom
Parts:
- added TP22, TP23, TP24, TP25: TestPoint, TestPoint:TestPoint_Pad_D2.0mm, symbol Connector:TestPoint
Connections:
- net at U507.1 (~{CS}), U508.39 (~{SPI_CS}): now also TP25.1
- net at U507.2 (MISO), U508.36 (SPI_POCI): now also TP24.1
- net at U507.5 (MOSI), U508.37 (SPI_PICO): now also TP23.1
- net at U507.6 (SCK), U508.38 (SPI_CLK): now also TP22.1
