File: io_banks.kicad_sch (KiCad schematic)
At the start: 27 parts, among them J25 AUX, J26 Conn_01x02, J27 PinHeader_2x22_P1.27mm, U22 ICE40HX8K-BG121, U26 SN74LVC1T45DCKR

Commit message: REV 0
Connections:
- net GND renamed GGND
Changed lines of the file:
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@@
 			)
 		)
-		(property "Value" "GND"
+		(property "Value" "GGND"
 			(at 80.01 85.09 0)
 			(effects
@@
 			)
 		)
-		(property "Value" "GND"
+		(property "Value" "GGND"
 			(at 109.347 72.9742 0)
 			(effects
@@
 			)
 		)
-		(property "Value" "GND"
+		(property "Value" "GGND"
 			(at 255.143 145.3642 0)
 			(effects
@@
 			)
 		)
-		(property "Value" "GND"
+		(property "Value" "GGND"
 			(at 254.127 52.6542 0)
 			(effects
@@
 			)
 		)
-		(property "Value" "GND"
+		(property "Value" "GGND"
 			(at 71.12 72.39 0)
 			(effects
@@
 			)
 		)
-		(property "Value" "GND"
+		(property "Value" "GGND"
 			(at 49.657 79.3242 0)
 			(effects
@@
 			)
 		)
-		(property "Value" "GND"
+		(property "Value" "GGND"
 			(at 53.34 57.15 0)
 			(effects
@@
 			)
 		)
-		(property "Value" "GND"
+		(property "Value" "GGND"
 			(at 59.69 119.38 90)
 			(effects
@@
 			)
 		)
-		(property "Value" "GND"
+		(property "Value" "GGND"
 			(at 221.107 70.4342 0)
 			(effects
@@
 			)
 		)
-		(property "Value" "GND"
+		(property "Value" "GGND"
 			(at 59.69 116.84 90)
 			(effects
@@
 			)
 		)
-		(property "Value" "GND"
+		(property "Value" "GGND"
 			(at 231.267 70.4342 0)
 			(effects
