File: io_buffer.kicad_sch (KiCad schematic)
At the start: 68 parts, among them J28 IDC-Header_2x10_P2.54mm, J29 Conn_01x08, J30 Conn_01x08, U27 SN74LVC1T45DCKR, U28 SN74LVC1T45DCKR, U29 SN74LVC1T45DCKR, U30 SN74LVC1T45DCKR, U31 SN74LVC1T45DCKR, U32 SN74LVC1T45DCKR, U33 SN74LVC1T45DCKR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

Commit message: REV 0
Connections:
- net GND renamed GGND
Changed lines of the file:
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@@
 			)
 		)
-		(property "Value" "GND"
+		(property "Value" "GGND"
 			(at 261.747 93.2942 0)
 			(effects
@@
 			)
 		)
-		(property "Value" "GND"
+		(property "Value" "GGND"
 			(at 249.047 118.6942 0)
 			(effects
@@
 			)
 		)
-		(property "Value" "GND"
+		(property "Value" "GGND"
 			(at 218.567 86.9442 0)
 			(effects
@@
 			)
 		)
-		(property "Value" "GND"
+		(property "Value" "GGND"
 			(at 254.127 37.4142 0)
 			(effects
@@
 			)
 		)
-		(property "Value" "GND"
+		(property "Value" "GGND"
 			(at 242.697 154.2542 0)
 			(effects
@@
 			)
 		)
-		(property "Value" "GND"
+		(property "Value" "GGND"
 			(at 233.807 53.9242 0)
 			(effects
@@
 			)
 		)
-		(property "Value" "GND"
+		(property "Value" "GGND"
 			(at 200.787 164.4142 0)
 			(effects
@@
 			)
 		)
-		(property "Value" "GND"
+		(property "Value" "GGND"
 			(at 278.257 163.1442 0)
 			(effects
@@
 			)
 		)
-		(property "Value" "GND"
+		(property "Value" "GGND"
 			(at 63.627 51.3842 0)
 			(effects
@@
 			)
 		)
-		(property "Value" "GND"
+		(property "Value" "GGND"
 			(at 50.927 34.8742 0)
 			(effects
@@
 			)
 		)
-		(property "Value" "GND"
+		(property "Value" "GGND"
 			(at 76.327 34.8742 0)
 			(effects
@@
 			)
 		)
-		(property "Value" "GND"
+		(property "Value" "GGND"
 			(at 63.627 92.0242 0)
 			(effects
@@
 			)
 		)
-		(property "Value" "GND"
+		(property "Value" "GGND"
 			(at 50.927 75.5142 0)
 			(effects
@@
 			)
 		)
-		(property "Value" "GND"
+		(property "Value" "GGND"
 			(at 76.327 75.5142 0)
 			(effects
@@
 			)
 		)
-		(property "Value" "GND"
+		(property "Value" "GGND"
 			(at 63.627 132.6642 0)
 			(effects
@@
 			)
 		)
-		(property "Value" "GND"
+		(property "Value" "GGND"
 			(at 50.927 116.1542 0)
 			(effects
@@
 			)
 		)
-		(property "Value" "GND"
+		(property "Value" "GGND"
 			(at 76.327 116.1542 0)
 			(effects
@@
 			)
 		)
-		(property "Value" "GND"
+		(property "Value" "GGND"
 			(at 63.627 173.3042 0)
 			(effects
@@
 			)
 		)
-		(property "Value" "GND"
+		(property "Value" "GGND"
 			(at 50.927 156.7942 0)
 			(effects
@@
 			)
 		)
-		(property "Value" "GND"
+		(property "Value" "GGND"
 			(at 76.327 156.7942 0)
 			(effects
@@
 			)
 		)
-		(property "Value" "GND"
+		(property "Value" "GGND"
 			(at 108.077 71.7042 0)
 			(effects
@@
 			)
 		)
-		(property "Value" "GND"
+		(property "Value" "GGND"
 			(at 95.377 55.1942 0)
 			(effects
@@
 			)
 		)
-		(property "Value" "GND"
+		(property "Value" "GGND"
 			(at 120.777 55.1942 0)
 			(effects
@@
 			)
 		)
-		(property "Value" "GND"
+		(property "Value" "GGND"
 			(at 108.077 112.3442 0)
 			(effects
@@
 			)
 		)
-		(property "Value" "GND"
+		(property "Value" "GGND"
 			(at 95.377 95.8342 0)
 			(effects
@@
 			)
 		)
-		(property "Value" "GND"
+		(property "Value" "GGND"
 			(at 120.777 95.8342 0)
 			(effects
@@
 			)
 		)
-		(property "Value" "GND"
+		(property "Value" "GGND"
 			(at 108.077 152.9842 0)
 			(effects
@@
 			)
 		)
-		(property "Value" "GND"
+		(property "Value" "GGND"
 			(at 95.377 136.4742 0)
 			(effects
@@
 			)
 		)
-		(property "Value" "GND"
+		(property "Value" "GGND"
 			(at 120.777 136.4742 0)
 			(effects
@@
 			)
 		)
-		(property "Value" "GND"
+		(property "Value" "GGND"
 			(at 108.077 193.6242 0)
 			(effects
@@
 			)
 		)
-		(property "Value" "GND"
+		(property "Value" "GGND"
 			(at 95.377 177.1142 0)
 			(effects
@@
 			)
 		)
-		(property "Value" "GND"
+		(property "Value" "GGND"
 			(at 120.777 177.1142 0)
 			(effects
@@
 			)
 		)
-		(property "Value" "GND"
+		(property "Value" "GGND"
 			(at 169.037 152.9842 0)
 			(effects
@@
 			)
 		)
-		(property "Value" "GND"
+		(property "Value" "GGND"
 			(at 174.117 114.8842 0)
 			(effects
@@
 			)
 		)
-		(property "Value" "GND"
+		(property "Value" "GGND"
 			(at 242.697 53.9242 0)
 			(effects
@@
 			)
 		)
-		(property "Value" "GND"
+		(property "Value" "GGND"
 			(at 161.417 114.8842 0)
 			(effects
@@
 			)
 		)
-		(property "Value" "GND"
+		(property "Value" "GGND"
 			(at 221.107 164.4142 0)
 			(effects
@@
 			)
 		)
-		(property "Value" "GND"
+		(property "Value" "GGND"
 			(at 271.907 152.9842 0)
 			(effects
@@
 			)
 		)
-		(property "Value" "GND"
+		(property "Value" "GGND"
 			(at 210.947 164.4142 0)
 			(effects
@@
 			)
 		)
-		(property "Value" "GND"
+		(property "Value" "GGND"
 			(at 219.837 53.9242 0)
 			(effects
@@
 			)
 		)
-		(property "Value" "GND"
+		(property "Value" "GGND"
 			(at 249.047 53.9242 0)
 			(effects
@@
 			)
 		)
-		(property "Value" "GND"
+		(property "Value" "GGND"
 			(at 146.177 22.1742 0)
 			(effects
@@
 			)
 		)
-		(property "Value" "GND"
+		(property "Value" "GGND"
 			(at 277.5712 67.183 90)
 			(effects
@@
 			)
 		)
-		(property "Value" "GND"
+		(property "Value" "GGND"
 			(at 226.187 81.8642 0)
 			(effects
