File: microcyber.kicad_sch (KiCad schematic)
At the start: 6 parts

Commit message: finished schematic draft and started placing components
Connections:
- no-connect marks 0 -> 3
Other:
- sheet Power_Supply renamed USBPD
- removed sheet Fan
- added sheet HDMI (HDMI.kicad_sch)
- added sheet PSU (PSU.kicad_sch)
- sheet Ethernet ports: added GbE_PCIe_CLK+, GbE_PCIe_CLK-, GbE_PCIe_RX+, GbE_PCIe_RX-, GbE_PCIe_TX+, GbE_PCIe_TX-, ~{CLKREQ4}, ~{PLT_RST}; removed none
- sheet M2_MKEY ports: added PCIE_RX_1+, PCIE_RX_1-, PCIE_TX_1+, PCIE_TX_1-, REFCLKM+, REFCLKM-, SUSCLK, ~{CLKREQM}, ~{PLT_RST}, ~{WAKE}; removed none
- sheet PCIEX4 ports: added PCIE_RX_0+, PCIE_RX_0-, PCIE_RX_1+, PCIE_RX_1-, PCIE_RX_2+, PCIE_RX_2-, PCIE_RX_3+, PCIE_RX_3-, PCIE_TX_0+, PCIE_TX_0-, PCIE_TX_1+, PCIE_TX_1-, PCIE_TX_2+, PCIE_TX_2-, PCIE_TX_3+, PCIE_TX_3-, REFCLK+, REFCLK-, ~{PLT_RST}, ~{WAKE}; removed none
- sheet USBPD: file Power_Supply.kicad_sch -> USBPD.kicad_sch
- sheet USBPD ports: added SUPPLY_GND, SUPPLY_PWR; removed none
- sheet USB_2_3 ports: added USB3_SSRX_N, USB3_SSRX_P, USB3_SSTX_N, USB3_SSTX_P, USB4_SSRX_N, USB4_SSRX_P, USB4_SSTX_N, USB4_SSTX_P, USB_2_P1+, USB_2_P1-, USB_2_P2+, USB_2_P2-, USB_2_P3+, USB_2_P3-, USB_2_P5+, USB_2_P5-, d1+_glas, d1-_glas, d2+_glas, d2-_glas, usb_gnd, vbus1_glas, vbus2_glas; removed none

Commit message: commit before removing duplicated glasgow
Parts:
- added TP28: PD_I2C0_SCL, TestPoint:TestPoint_Pad_2.5x2.5mm, symbol Connector:TestPoint
- added TP29: PD_I2C0_SDA, TestPoint:TestPoint_Pad_2.5x2.5mm, symbol Connector:TestPoint
- added TP30: PD_I2C1_SCL, TestPoint:TestPoint_Pad_2.5x2.5mm, symbol Connector:TestPoint
- added TP31: PD_I2C1_SDA, TestPoint:TestPoint_Pad_2.5x2.5mm, symbol Connector:TestPoint
- FID1, FID2: footprint (none) -> Fiducial:Fiducial_1.5mm_Mask3mm
- H1, H4: footprint (none) -> MountingHole:MountingHole_2.7mm_Pad_TopOnly
- H2: renamed from H3; footprint (none) -> MountingHole:MountingHole_2.7mm_Pad_TopOnly
- H3: renamed from H2; footprint (none) -> MountingHole:MountingHole_2.7mm_Pad_TopOnly
Connections:
- new net USBPD/PD_I2C0_SCL: TP28.1
- new net USBPD/PD_I2C0_SDA: TP29.1
- new net USBPD/PD_I2C1_SCL: TP30.1
- new net USBPD/PD_I2C1_SDA: TP31.1
- no-connect marks 3 -> 2
Other:
- removed sheet PCIEX4
- added sheet M2_EKEY (M2_EKEY.kicad_sch)
- added sheet extendoboard (extendo.kicad_sch)
- sheet GPIO ports: added none; removed I2C5_SCL, I2C5_SDA
- sheet LattePanda_Module ports: added CLKREQ3, CLKREQ4, REFCLK1+, REFCLK1-, USB_2_P4+, USB_2_P4-, USB_2_P8+, USB_2_P8-; removed USB_2_P6+, USB_2_P6-
- sheet USBPD ports: added BATT_GND, BATT_SUPPLY, PD_I2C0_SCL, PD_I2C0_SDA, PD_I2C1_SCL, PD_I2C1_SDA, VBUS_POWER; removed none
- sheet USB_2_3 ports: added none; removed USB_2_P3+, USB_2_P3-, d2+_glas, d2-_glas
- sheet glasgow ports: added SCL, SDA; removed none

Commit message: before board exclusion
Changed lines of the file:
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@@
 	)
 	(junction
-		(at 123.19 26.67)
-		(diameter 0)
-		(color 0 0 0 0)
-	)
-	(junction
-		(at 123.19 30.48)
-		(diameter 0)
-		(color 0 0 0 0)
-	)
-	(junction
 		(at 425.45 334.01)
 		(diameter 0)
@@
 	(wire
 		(pts
-			(xy 123.19 30.48) (xy 123.19 26.67)
-		)
-		(stroke
-			(width 0)
-			(type default)
-		)
-	)
-	(wire
-		(pts
 			(xy 158.75 168.91) (xy 177.8 168.91)
 		)
@@
 	(wire
 		(pts
-			(xy 82.55 71.12) (xy 87.63 71.12)
-		)
-		(stroke
-			(width 0)
-			(type default)
-		)
-	)
-	(wire
-		(pts
 			(xy 127 73.66) (xy 127 93.98)
 		)
@@
 	(wire
 		(pts
+			(xy 82.55 73.66) (xy 92.71 73.66)
+		)
+		(stroke
+			(width 0)
+			(type default)
+		)
+	)
+	(wire
+		(pts
 			(xy 158.75 186.69) (xy 189.23 186.69)
 		)
@@
 	(wire
 		(pts
+			(xy 92.71 30.48) (xy 92.71 73.66)
+		)
+		(stroke
+			(width 0)
+			(type default)
+		)
+	)
+	(wire
+		(pts
 			(xy 331.47 243.84) (xy 347.98 243.84)
 		)
@@
 	(wire
 		(pts
+			(xy 82.55 69.85) (xy 87.63 69.85)
+		)
+		(stroke
+			(width 0)
+			(type default)
+		)
+	)
+	(wire
+		(pts
 			(xy 331.47 229.87) (xy 347.98 229.87)
 		)
@@
 	(wire
 		(pts
-			(xy 87.63 26.67) (xy 87.63 71.12)
+			(xy 87.63 26.67) (xy 87.63 69.85)
 		)
 		(stroke
@@
 	(wire
 		(pts
-			(xy 104.14 30.48) (xy 123.19 30.48)
-		)
-		(stroke
-			(width 0)
-			(type default)
-		)
-	)
-	(wire
-		(pts
 			(xy 407.67 317.5) (xy 429.26 317.5)
 		)
@@
 	(wire
 		(pts
-			(xy 104.14 30.48) (xy 104.14 77.47)
-		)
-		(stroke
-			(width 0)
-			(type default)
-		)
-	)
-	(wire
-		(pts
 			(xy 331.47 318.77) (xy 345.44 318.77)
 		)
@@
 	(wire
 		(pts
-			(xy 445.77 336.55) (xy 425.45 336.55)
+			(xy 92.71 30.48) (xy 123.19 30.48)
 		)
 		(stroke
@@
 	(wire
 		(pts
-			(xy 104.14 77.47) (xy 82.55 77.47)
+			(xy 445.77 336.55) (xy 425.45 336.55)
 		)
 		(stroke
@@
 		(in_bom yes)
 		(on_board yes)
-		(dnp no)
+		(dnp yes)
 		(fields_autoplaced yes)
 		(stroke
@@
 		(in_bom yes)
 		(on_board yes)
-		(dnp no)
+		(dnp yes)
 		(fields_autoplaced yes)
 		(stroke
@@
 		)
 		(pin "SUPPLY_GND" input
-			(at 82.55 77.47 0)
+			(at 82.55 69.85 0)
 			(effects
 				(font
@@
 		)
 		(pin "SUPPLY_PWR" input
-			(at 82.55 71.12 0)
+			(at 82.55 73.66 0)
 			(effects
 				(font

Commit message: REV 0
Parts:
- added NT3: NetTie_2, NetTie:NetTie-2_THT_Pad1.0mm, symbol Device:NetTie_2
- added R152, R153: 0, Resistor_SMD:R_0612_1632Metric_Pad1.18x3.40mm_HandSolder, symbol Library:R
- TP28, TP29, TP30, TP31: now not fitted
Connections:
- net LattePanda_Module/I2C5_SCL: now also R152.1
- net LattePanda_Module/I2C5_SDA: now also R153.1
- net USB_2_3/usb_gnd: now also NT3.1
- new net glasgow/GND: NT3.2
- new net glasgow/SCL: R152.2
- new net glasgow/SDA: R153.2
Other:
- sheet PSU ports: added EDGEBOARD_GND, EDGEBOARD_SUPPLY; removed none
