File: glasgow.kicad_sch (KiCad schematic)
At the start: 92 parts, among them SW1 RST, U18 TPD3S014, U19 CY7C68013A-56LTX, U20 CAT24M01X, U21 BL24C256A-SFRC, U22 ICE40HX8K-BG121, U23 APX811-40UG-7, U24 TLV75533PDRVR, U25 TLV73312PQDRVR, Y2 24M

Commit message: went back to the drawing board
Parts:
- removed MK1, MK2: Mounting_Hole_PAD, Glasgow:MountingHole_3.5mm_Pad_Via_CrtYd, symbol Mechanical:MountingHole_Pad

Commit message: V4 done ???
Parts:
- C94, R41: now not fitted; now left out of the parts list
Changed lines of the file:
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@@
 		(body_style 1)
 		(exclude_from_sim no)
-		(in_bom yes)
-		(on_board yes)
-		(in_pos_files yes)
-		(dnp no)
+		(in_bom no)
+		(on_board no)
+		(in_pos_files yes)
+		(dnp yes)
 		(property "Reference" "R41"
 			(at 29.21 161.29 0)
@@
 		(body_style 1)
 		(exclude_from_sim no)
-		(in_bom yes)
-		(on_board yes)
-		(in_pos_files yes)
-		(dnp no)
+		(in_bom no)
+		(on_board no)
+		(in_pos_files yes)
+		(dnp yes)
 		(property "Reference" "C94"
 			(at 21.971 160.1216 0)
