File: rpi.kicad_sch (KiCad schematic)
At the start: 1 part

Commit message: rpi edgeboard
Connections:
- net GPIO_8: now reaches A2.20 (GPIO15)
- net GPIO_1: now reaches A2.21 (GPIO16)
- net GPIO_2: now reaches A2.22 (GPIO17)
- net GPIO_3: now reaches A2.24 (GPIO18)
- net GPIO_4: now reaches A2.25 (GPIO19)
- net GPIO_5: now reaches A2.26 (GPIO20)
- net GPIO_6: now reaches A2.27 (GPIO21)
- net GPIO_7: now reaches A2.29 (GPIO22)
Changed lines of the file:
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@@
 	(generator_version "10.0")
 	(paper "A4")
+	(label "GPIO_6"
+		(at 0.1588 2.0957 0)
+		(effects
+			(font
+				(size 1.27 1.27)
+			)
+			(justify left bottom)
+		)
+	)
+	(label "GPIO_6"
+		(at 2.6988 4.6357 0)
+		(effects
+			(font
+				(size 1.27 1.27)
+			)
+			(justify left bottom)
+		)
+	)
 	(hierarchical_label "I2C0_SCL"
 		(shape input)
@@
 			)
 			(justify right)
+		)
+	)
+	(hierarchical_label "GPIO_2"
+		(shape input)
+		(at 168.91 69.85 0)
+		(effects
+			(font
+				(size 1.27 1.27)
+			)
+			(justify left)
 		)
 	)
@@
 		)
 	)
+	(hierarchical_label "GPIO_5"
+		(shape input)
+		(at 168.91 77.47 0)
+		(effects
+			(font
+				(size 1.27 1.27)
+			)
+			(justify left)
+		)
+	)
 	(hierarchical_label "SPIO0_RX"
 		(shape input)
@@
 			)
 			(justify right)
+		)
+	)
+	(hierarchical_label "GPIO_1"
+		(shape input)
+		(at 168.91 67.31 0)
+		(effects
+			(font
+				(size 1.27 1.27)
+			)
+			(justify left)
 		)
 	)
@@
 		)
 	)
+	(hierarchical_label "GPIO_6"
+		(shape input)
+		(at 168.91 80.01 0)
+		(effects
+			(font
+				(size 1.27 1.27)
+			)
+			(justify left)
+		)
+	)
+	(hierarchical_label "GPIO_4"
+		(shape input)
+		(at 168.91 74.93 0)
+		(effects
+			(font
+				(size 1.27 1.27)
+			)
+			(justify left)
+		)
+	)
+	(hierarchical_label "GPIO_3"
+		(shape input)
+		(at 168.91 72.39 0)
+		(effects
+			(font
+				(size 1.27 1.27)
+			)
+			(justify left)
+		)
+	)
 	(hierarchical_label "I2C1_SDA"
 		(shape input)
 		(at 123.19 80.01 180)
+		(effects
+			(font
+				(size 1.27 1.27)
+			)
+			(justify right)
+		)
+	)
+	(hierarchical_label "GPIO_8"
+		(shape input)
+		(at 123.19 102.87 180)
 		(effects
 			(font
@@
 		)
 	)
+	(hierarchical_label "GPIO_7"
+		(shape input)
+		(at 168.91 82.55 0)
+		(effects
+			(font
+				(size 1.27 1.27)
+			)
+			(justify left)
+		)
+	)

Commit message: V4 done ???
Parts:
- A2: footprint Module:RaspberryPi_Pico_SMD_HandSolder -> Module:RaspberryPi_Pico_Common_THT
Changed lines of the file:
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@@
 			)
 		)
-		(property "Footprint" "Module:RaspberryPi_Pico_SMD_HandSolder"
+		(property "Footprint" "Module:RaspberryPi_Pico_Common_THT"
 			(at 146.05 127 0)
 			(hide yes)

Commit message: hdmi diff pair remains??
Parts:
- added J5: Conn_01x01_Socket, Connector_PinHeader_2.00mm:PinHeader_1x01_P2.00mm_Horizontal, symbol Connector:Conn_01x01_Socket
Connections:
- net +5V: no longer names the net of A2.39 (VSYS)
- net +5V: now also J5.1 (Pin_1)
Changed lines of the file:
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@@
 	)
 	(symbol
-		(lib_id "power:+5V")
-		(at 140.97 41.91 0)
+		(lib_id "Connector:Conn_01x01_Socket")
+		(at 140.97 36.83 90)
 		(unit 1)
 		(body_style 1)
@@
 		(in_pos_files yes)
 		(dnp no)
-		(fields_autoplaced yes)
-		(property "Reference" "#PWR0246"
-			(at 140.97 45.72 0)
-			(hide yes)
+		(property "Reference" "J5"
+			(at 139.6999 35.56 0)
 			(show_name no)
 			(do_not_autoplace no)
@@
 					(size 1.27 1.27)
 				)
+				(justify left)
 			)
 		)
-		(property "Value" "+5V"
-			(at 140.97 36.83 0)
+		(property "Value" "Conn_01x01_Socket"
+			(at 140.462 34.29 0)
 			(show_name no)
 			(do_not_autoplace no)
@@
 					(size 1.27 1.27)
 				)
+				(justify left)
 			)
 		)
-		(property "Footprint" ""
-			(at 140.97 41.91 0)
+		(property "Footprint" "Connector_PinHeader_2.00mm:PinHeader_1x01_P2.00mm_Horizontal"
+			(at 131.572 34.544 0)
 			(hide yes)
 			(show_name no)
@@
 		)
 		(property "Datasheet" ""
-			(at 140.97 41.91 0)
+			(at 140.97 36.83 0)
 			(hide yes)
 			(show_name no)
@@
 			)
 		)
-		(property "Description" "Power symbol creates a global label with name \"+5V\""
-			(at 140.97 41.91 0)
+		(property "Description" "Generic connector, single row, 01x01, script generated"
+			(at 140.97 36.83 0)
 			(hide yes)
 			(show_name no)
@@
 			(project "microcyber"
 				(path "/7ac319af-771c-4997-a005-b73a4a9b44ab/4c3faca8-bed6-416d-8c17-d21c07d6704e"
-					(reference "#PWR0246")
+					(reference "J5")
 					(unit 1)
 				)
