File: GPIO.kicad_sch (KiCad schematic)
At the start: 16 parts, among them J10 Conn_01x03_Pin, J11 Conn_01x03_Pin, J12 Conn_01x04_Pin, J13 Conn_01x04_Pin, J14 Conn_01x03_Pin, J19 Conn_01x04_Pin, J20 Conn_01x04_Pin, J21 Conn_01x04_Pin, J7 Conn_01x04_Pin, J8 Conn_01x03_Pin, J9 Conn_01x04_Pin, U1 ULC0524P, U10 ULC0524P, U11 ULC0524P, U12 ULC0524P, U9 ULC0524P

Commit message: commit before removing duplicated glasgow
Parts:
- renumbered J7 to J10, J8 to J11, J10 to J12, J9 to J13, J12 to J14, J11 to J15, J13 to J16, J14 to J17, J19 to J18, J20 to J19, J21 to J20, U1 to U11, U9 to U7, U11 to U8, U12 to U9
Changed lines of the file:
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@@
-		)
-	)
-	(hierarchical_label "I2C5_SCL"
-		(shape output)
-		(at 181.61 45.72 0)
-		(effects
-			(font
-				(size 1.27 1.27)
-			)
-			(justify left)
 		)
 	)
@@
 		)
 	)
-	(hierarchical_label "I2C5_SDA"
-		(shape bidirectional)
-		(at 71.12 38.1 0)
-		(effects
-			(font
-				(size 1.27 1.27)
-			)
-			(justify left)
-		)
-	)
 	(hierarchical_label "SOC_UART0_TX"
 		(shape input)
@@
 		(dnp no)
 		(fields_autoplaced yes)
-		(property "Reference" "U1"
+		(property "Reference" "U11"
 			(at 257.81 72.39 0)
 			(effects
@@
 			(project "microcyber"
 				(path "/7ac319af-771c-4997-a005-b73a4a9b44ab/46baeb5e-c32d-4e80-9378-f9d622006dfc"
-					(reference "U1")
+					(reference "U11")
 					(unit 1)
 				)
@@
 		(dnp no)
 		(fields_autoplaced yes)
-		(property "Reference" "#PWR023"
+		(property "Reference" "#PWR061"
 			(at 252.73 128.27 0)
 			(effects
@@
 			(project ""
 				(path "/7ac319af-771c-4997-a005-b73a4a9b44ab/46baeb5e-c32d-4e80-9378-f9d622006dfc"
-					(reference "#PWR023")
+					(reference "#PWR061")
 					(unit 1)
 				)
@@
 		(dnp no)
 		(fields_autoplaced yes)
-		(property "Reference" "J13"
+		(property "Reference" "J16"
 			(at 222.885 33.02 0)
 			(effects
@@
 			(project "microcyber"
 				(path "/7ac319af-771c-4997-a005-b73a4a9b44ab/46baeb5e-c32d-4e80-9378-f9d622006dfc"
-					(reference "J13")
+					(reference "J16")
 					(unit 1)
 				)
@@
 		(dnp no)
 		(fields_autoplaced yes)
-		(property "Reference" "J10"
+		(property "Reference" "J12"
 			(at 103.505 97.79 0)
 			(effects
@@
 			(project "microcyber"
 				(path "/7ac319af-771c-4997-a005-b73a4a9b44ab/46baeb5e-c32d-4e80-9378-f9d622006dfc"
-					(reference "J10")
+					(reference "J12")
 					(unit 1)
 				)
@@
 		(dnp no)
 		(fields_autoplaced yes)
-		(property "Reference" "#PWR022"
+		(property "Reference" "#PWR054"
 			(at 52.07 146.05 0)
 			(effects
@@
 			(project "microcyber"
 				(path "/7ac319af-771c-4997-a005-b73a4a9b44ab/46baeb5e-c32d-4e80-9378-f9d622006dfc"
-					(reference "#PWR022")
+					(reference "#PWR054")
 					(unit 1)
 				)
@@
 		(dnp no)
 		(fields_autoplaced yes)
-		(property "Reference" "#PWR021"
+		(property "Reference" "#PWR055"
 			(at 134.62 144.78 0)
 			(effects
@@
 			(project ""
 				(path "/7ac319af-771c-4997-a005-b73a4a9b44ab/46baeb5e-c32d-4e80-9378-f9d622006dfc"
-					(reference "#PWR021")
+					(reference "#PWR055")
 					(unit 1)
 				)
@@
 		(dnp no)
 		(fields_autoplaced yes)
-		(property "Reference" "#PWR019"
+		(property "Reference" "#PWR058"
 			(at 209.55 113.03 0)
 			(effects
@@
 			(project ""
 				(path "/7ac319af-771c-4997-a005-b73a4a9b44ab/46baeb5e-c32d-4e80-9378-f9d622006dfc"
-					(reference "#PWR019")
+					(reference "#PWR058")
 					(unit 1)
 				)
@@
 		(dnp no)
 		(fields_autoplaced yes)
-		(property "Reference" "J7"
+		(property "Reference" "J10"
 			(at 41.275 25.4 0)
 			(effects
@@
 			(project ""
 				(path "/7ac319af-771c-4997-a005-b73a4a9b44ab/46baeb5e-c32d-4e80-9378-f9d622006dfc"
-					(reference "J7")
+					(reference "J10")
 					(unit 1)
 				)
@@
 		(dnp no)
 		(fields_autoplaced yes)
-		(property "Reference" "J12"
+		(property "Reference" "J14"
 			(at 196.215 31.75 0)
 			(effects
@@
 			(project "microcyber"
 				(path "/7ac319af-771c-4997-a005-b73a4a9b44ab/46baeb5e-c32d-4e80-9378-f9d622006dfc"
-					(reference "J12")
+					(reference "J14")
 					(unit 1)
 				)
@@
 		(dnp no)
 		(fields_autoplaced yes)
-		(property "Reference" "#PWR018"
+		(property "Reference" "#PWR053"
 			(at 52.07 92.71 0)
 			(effects
@@
 			(project "microcyber"
 				(path "/7ac319af-771c-4997-a005-b73a4a9b44ab/46baeb5e-c32d-4e80-9378-f9d622006dfc"
-					(reference "#PWR018")
+					(reference "#PWR053")
 					(unit 1)
 				)
@@
 		(dnp no)
 		(fields_autoplaced yes)
-		(property "Reference" "J9"
+		(property "Reference" "J13"
 			(at 153.035 33.02 0)
 			(effects
@@
 			(project "microcyber"
 				(path "/7ac319af-771c-4997-a005-b73a4a9b44ab/46baeb5e-c32d-4e80-9378-f9d622006dfc"
-					(reference "J9")
+					(reference "J13")
 					(unit 1)
 				)
@@
 		(dnp no)
 		(fields_autoplaced yes)
-		(property "Reference" "#PWR024"
+		(property "Reference" "#PWR063"
 			(at 275.59 116.84 0)
 			(effects
@@
 			(project ""
 				(path "/7ac319af-771c-4997-a005-b73a4a9b44ab/46baeb5e-c32d-4e80-9378-f9d622006dfc"
-					(reference "#PWR024")
+					(reference "#PWR063")
 					(unit 1)
 				)
@@
 		(dnp no)
 		(fields_autoplaced yes)
-		(property "Reference" "#PWR015"
+		(property "Reference" "#PWR057"
 			(at 200.66 54.61 0)
 			(effects
@@
 			(project ""
 				(path "/7ac319af-771c-4997-a005-b73a4a9b44ab/46baeb5e-c32d-4e80-9378-f9d622006dfc"
-					(reference "#PWR015")
+					(reference "#PWR057")
 					(unit 1)
 				)
@@
 		(dnp no)
 		(fields_autoplaced yes)
-		(property "Reference" "#PWR017"
+		(property "Reference" "#PWR056"
 			(at 135.89 92.71 0)
 			(effects
@@
 			(project ""
 				(path "/7ac319af-771c-4997-a005-b73a4a9b44ab/46baeb5e-c32d-4e80-9378-f9d622006dfc"
-					(reference "#PWR017")
+					(reference "#PWR056")
 					(unit 1)
 				)
@@
 		(dnp no)
 		(fields_autoplaced yes)
-		(property "Reference" "#PWR016"
+		(property "Reference" "#PWR059"
 			(at 233.68 41.91 0)
 			(effects
@@
 			(project ""
 				(path "/7ac319af-771c-4997-a005-b73a4a9b44ab/46baeb5e-c32d-4e80-9378-f9d622006dfc"
-					(reference "#PWR016")
+					(reference "#PWR059")
 					(unit 1)
 				)
@@
 		(dnp no)
 		(fields_autoplaced yes)
-		(property "Reference" "#PWR020"
+		(property "Reference" "#PWR060"
 			(at 236.22 102.87 0)
 			(effects
@@
 			(project ""
 				(path "/7ac319af-771c-4997-a005-b73a4a9b44ab/46baeb5e-c32d-4e80-9378-f9d622006dfc"
-					(reference "#PWR020")
+					(reference "#PWR060")
 					(unit 1)
 				)
@@
 		(dnp no)
 		(fields_autoplaced yes)
-		(property "Reference" "U12"
+		(property "Reference" "U9"
 			(at 134.62 113.03 0)
 			(effects
@@
 			(project "microcyber"
 				(path "/7ac319af-771c-4997-a005-b73a4a9b44ab/46baeb5e-c32d-4e80-9378-f9d622006dfc"
-					(reference "U12")
+					(reference "U9")
 					(unit 1)
 				)
@@
 		(dnp no)
 		(fields_autoplaced yes)
-		(property "Reference" "U9"
+		(property "Reference" "U7"
 			(at 52.07 60.96 0)
 			(effects
@@
 			(project ""
 				(path "/7ac319af-771c-4997-a005-b73a4a9b44ab/46baeb5e-c32d-4e80-9378-f9d622006dfc"
-					(reference "U9")
+					(reference "U7")
 					(unit 1)
 				)
@@
 		(dnp no)
 		(fields_autoplaced yes)
-		(property "Reference" "J11"
+		(property "Reference" "J15"
 			(at 205.105 93.98 0)
 			(effects
@@
 			(project "microcyber"
 				(path "/7ac319af-771c-4997-a005-b73a4a9b44ab/46baeb5e-c32d-4e80-9378-f9d622006dfc"
-					(reference "J11")
+					(reference "J15")
 					(unit 1)
 				)
@@
 		(dnp no)
 		(fields_autoplaced yes)
-		(property "Reference" "J8"
+		(property "Reference" "J11"
 			(at 47.625 99.06 0)
 			(effects
@@
 			(project "microcyber"
 				(path "/7ac319af-771c-4997-a005-b73a4a9b44ab/46baeb5e-c32d-4e80-9378-f9d622006dfc"
-					(reference "J8")
+					(reference "J11")
 					(unit 1)
 				)
@@
 		(dnp no)
 		(fields_autoplaced yes)
-		(property "Reference" "J20"
+		(property "Reference" "J19"
 			(at 248.285 106.68 0)
 			(effects
@@
 			(project "microcyber"
 				(path "/7ac319af-771c-4997-a005-b73a4a9b44ab/46baeb5e-c32d-4e80-9378-f9d622006dfc"
-					(reference "J20")
+					(reference "J19")
 					(unit 1)
 				)
@@
 		(dnp no)
 		(fields_autoplaced yes)
-		(property "Reference" "J14"
+		(property "Reference" "J17"
 			(at 225.425 93.98 0)
 			(effects
@@
 			(project "microcyber"
 				(path "/7ac319af-771c-4997-a005-b73a4a9b44ab/46baeb5e-c32d-4e80-9378-f9d622006dfc"
-					(reference "J14")
+					(reference "J17")
 					(unit 1)
 				)
@@
 		(dnp no)
 		(fields_autoplaced yes)
-		(property "Reference" "#PWR025"
+		(property "Reference" "#PWR062"
 			(at 257.81 104.14 0)
 			(effects
@@
 			(project ""
 				(path "/7ac319af-771c-4997-a005-b73a4a9b44ab/46baeb5e-c32d-4e80-9378-f9d622006dfc"
-					(reference "#PWR025")
+					(reference "#PWR062")
 					(unit 1)
 				)
@@
 		(dnp no)
 		(fields_autoplaced yes)
-		(property "Reference" "U11"
+		(property "Reference" "U8"
 			(at 52.07 114.3 0)
 			(effects
@@
 			(project "microcyber"
 				(path "/7ac319af-771c-4997-a005-b73a4a9b44ab/46baeb5e-c32d-4e80-9378-f9d622006dfc"
-					(reference "U11")
+					(reference "U8")
 					(unit 1)
 				)
@@
 		(dnp no)
 		(fields_autoplaced yes)
-		(property "Reference" "J19"
+		(property "Reference" "J18"
 			(at 231.775 49.53 0)
 			(effects
@@
 			(project "microcyber"
 				(path "/7ac319af-771c-4997-a005-b73a4a9b44ab/46baeb5e-c32d-4e80-9378-f9d622006dfc"
-					(reference "J19")
+					(reference "J18")
 					(unit 1)
 				)
@@
 		(dnp no)
 		(fields_autoplaced yes)
-		(property "Reference" "J21"
+		(property "Reference" "J20"
 			(at 266.065 107.95 0)
 			(effects
@@
 			(project "microcyber"
 				(path "/7ac319af-771c-4997-a005-b73a4a9b44ab/46baeb5e-c32d-4e80-9378-f9d622006dfc"
-					(reference "J21")
-					(unit 1)
-				)
+					(reference "J20")
+					(unit 1)
+				)

Commit message: is this a differential pair?
Parts:
- J10, J13, J14, J16, J18, J19, J20: DF_Comment (none) -> 2.54绿色单排排针-4P
- J11, J12, J15, J17: DF_Comment (none) -> 2.54红色单排排针-3P
Changed lines of the file:
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@@
+			)
+		)
+		(property "DF_Comment" "2.54绿色单排排针-4P"
+			(at 222.25 40.64 0)
+			(effects
+				(font
+					(size 1.27 1.27)
+				)
+				(hide yes)
+			)
+		)
+		(property "Field-1" ""
+			(at 222.25 40.64 0)
+			(effects
+				(font
+					(size 1.27 1.27)
+				)
+				(hide yes)
 			)
 		)
@@
 			)
 		)
+		(property "DF_Comment" "2.54红色单排排针-3P"
+			(at 102.87 105.41 0)
+			(effects
+				(font
+					(size 1.27 1.27)
+				)
+				(hide yes)
+			)
+		)
+		(property "Field-1" ""
+			(at 102.87 105.41 0)
+			(effects
+				(font
+					(size 1.27 1.27)
+				)
+				(hide yes)
+			)
+		)
 		(pin "2"
 		)
@@
 			)
 		)
+		(property "DF_Comment" "2.54绿色单排排针-4P"
+			(at 40.64 33.02 0)
+			(effects
+				(font
+					(size 1.27 1.27)
+				)
+				(hide yes)
+			)
+		)
+		(property "Field-1" ""
+			(at 40.64 33.02 0)
+			(effects
+				(font
+					(size 1.27 1.27)
+				)
+				(hide yes)
+			)
+		)
 		(pin "3"
 		)
@@
 			)
 		)
+		(property "DF_Comment" "2.54绿色单排排针-4P"
+			(at 195.58 39.37 0)
+			(effects
+				(font
+					(size 1.27 1.27)
+				)
+				(hide yes)
+			)
+		)
+		(property "Field-1" ""
+			(at 195.58 39.37 0)
+			(effects
+				(font
+					(size 1.27 1.27)
+				)
+				(hide yes)
+			)
+		)
 		(pin "3"
 		)
@@
 			)
 		)
+		(property "DF_Comment" "2.54绿色单排排针-4P"
+			(at 152.4 40.64 0)
+			(effects
+				(font
+					(size 1.27 1.27)
+				)
+				(hide yes)
+			)
+		)
+		(property "Field-1" ""
+			(at 152.4 40.64 0)
+			(effects
+				(font
+					(size 1.27 1.27)
+				)
+				(hide yes)
+			)
+		)
 		(pin "3"
 		)
@@
 			)
 		)
+		(property "DF_Comment" "2.54红色单排排针-3P"
+			(at 204.47 101.6 0)
+			(effects
+				(font
+					(size 1.27 1.27)
+				)
+				(hide yes)
+			)
+		)
+		(property "Field-1" ""
+			(at 204.47 101.6 0)
+			(effects
+				(font
+					(size 1.27 1.27)
+				)
+				(hide yes)
+			)
+		)
 		(pin "2"
 		)
@@
 			)
 		)
+		(property "DF_Comment" "2.54红色单排排针-3P"
+			(at 46.99 106.68 0)
+			(effects
+				(font
+					(size 1.27 1.27)
+				)
+				(hide yes)
+			)
+		)
+		(property "Field-1" ""
+			(at 46.99 106.68 0)
+			(effects
+				(font
+					(size 1.27 1.27)
+				)
+				(hide yes)
+			)
+		)
 		(pin "2"
 		)
@@
 			)
 		)
+		(property "DF_Comment" "2.54绿色单排排针-4P"
+			(at 247.65 114.3 0)
+			(effects
+				(font
+					(size 1.27 1.27)
+				)
+				(hide yes)
+			)
+		)
+		(property "Field-1" ""
+			(at 247.65 114.3 0)
+			(effects
+				(font
+					(size 1.27 1.27)
+				)
+				(hide yes)
+			)
+		)
 		(pin "3"
 		)
@@
 			)
 		)
+		(property "DF_Comment" "2.54红色单排排针-3P"
+			(at 224.79 101.6 0)
+			(effects
+				(font
+					(size 1.27 1.27)
+				)
+				(hide yes)
+			)
+		)
+		(property "Field-1" ""
+			(at 224.79 101.6 0)
+			(effects
+				(font
+					(size 1.27 1.27)
+				)
+				(hide yes)
+			)
+		)
 		(pin "2"
 		)
@@
 			)
 		)
+		(property "DF_Comment" "2.54绿色单排排针-4P"
+			(at 231.14 57.15 0)
+			(effects
+				(font
+					(size 1.27 1.27)
+				)
+				(hide yes)
+			)
+		)
+		(property "Field-1" ""
+			(at 231.14 57.15 0)
+			(effects
+				(font
+					(size 1.27 1.27)
+				)
+				(hide yes)
+			)
+		)
 		(pin "3"
 		)
@@
 			(at 265.43 115.57 0)
 			(effects
+				(font
+					(size 1.27 1.27)
+				)
+				(hide yes)
+			)
+		)
+		(property "DF_Comment" "2.54绿色单排排针-4P"
+			(at 265.43 115.57 0)
+			(effects
+				(font
+					(size 1.27 1.27)
+				)
+				(hide yes)
+			)
+		)
+		(property "Field-1" ""
+			(at 265.43 115.57 0)
+			(effects

Commit message: all power, diff pairs done, all components placed (final spot?) just some small wires left to route
Parts:
- removed J13, J14, J16, J19, J20: Conn_01x04_Pin, A_HDJ_Library:PinHeader_1x04_P2.54mm_Vertical, symbol Connector:Conn_01x04_Pin
Connections:
- net I2C2_SCL: now also J10.2 (Pin_2)
- net I2C3_SCL: no longer names the net of U10.2, U10.9 (NC)
- net I2C3_SDA: no longer names the net of U7.2, U7.9 (NC)
- net I2C3_SDA: no longer J10.2 (Pin_2)
- net I2C4_SCL: no longer names the net of U10.4, U10.7 (NC)
- net I2C4_SDA: no longer names the net of U7.4, U7.7 (NC)
- net I2C4_SDA: no longer J10.3 (Pin_3)
- net I2C5_SCL: no longer names the net of U10.5, U10.6 (NC)
- net I2C5_SDA: no longer names the net of U7.5, U7.6 (NC)
- net I2C5_SDA: no longer J10.4 (Pin_4)

Commit message: last push before editing with the grid view (gonna break everything)
Parts:
- J10, J11, J12, J15, J17, J18: now left out of the parts list
- U10, U11, U7, U8, U9: MPN (none) -> ULC0524P
Changed lines of the file:
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@@
+			)
+		)
+		(property "MPN" "ULC0524P"
+			(at 257.81 85.09 0)
+			(hide yes)
+			(show_name no)
+			(do_not_autoplace no)
+			(effects
+				(font
+					(size 1.27 1.27)
+				)
 			)
 		)
@@
 		(body_style 1)
 		(exclude_from_sim no)
-		(in_bom yes)
+		(in_bom no)
 		(on_board yes)
 		(in_pos_files yes)
@@
 		(body_style 1)
 		(exclude_from_sim no)
-		(in_bom yes)
+		(in_bom no)
 		(on_board yes)
 		(in_pos_files yes)
@@
 			)
 		)
+		(property "MPN" "ULC0524P"
+			(at 135.89 73.66 0)
+			(hide yes)
+			(show_name no)
+			(do_not_autoplace no)
+			(effects
+				(font
+					(size 1.27 1.27)
+				)
+			)
+		)
 		(pin "6"
 		)
@@
 			)
 		)
+		(property "MPN" "ULC0524P"
+			(at 134.62 125.73 0)
+			(hide yes)
+			(show_name no)
+			(do_not_autoplace no)
+			(effects
+				(font
+					(size 1.27 1.27)
+				)
+			)
+		)
 		(pin "6"
 		)
@@
 			)
 		)
+		(property "MPN" "ULC0524P"
+			(at 52.07 73.66 0)
+			(hide yes)
+			(show_name no)
+			(do_not_autoplace no)
+			(effects
+				(font
+					(size 1.27 1.27)
+				)
+			)
+		)
 		(pin "6"
 		)
@@
 		(body_style 1)
 		(exclude_from_sim no)
-		(in_bom yes)
+		(in_bom no)
 		(on_board yes)
 		(in_pos_files yes)
@@
 		(body_style 1)
 		(exclude_from_sim no)
-		(in_bom yes)
+		(in_bom no)
 		(on_board yes)
 		(in_pos_files yes)
@@
 		(body_style 1)
 		(exclude_from_sim no)
-		(in_bom yes)
+		(in_bom no)
 		(on_board yes)
 		(in_pos_files yes)
@@
 			)
 		)
+		(property "MPN" "ULC0524P"
+			(at 52.07 127 0)
+			(hide yes)
+			(show_name no)
+			(do_not_autoplace no)
+			(effects
+				(font
+					(size 1.27 1.27)
+				)
+			)
+		)
 		(pin "6"
 		)
@@
 		(body_style 1)
 		(exclude_from_sim no)
-		(in_bom yes)
-		(on_board yes)
-		(in_pos_files yes)
+		(in_bom no)
+		(on_board yes)
+		(in_pos_files yes)
