File: Ethernet.kicad_sch (KiCad schematic)
At the start: 0 parts

Commit message: finished schematic draft and started placing components
Parts:
- added C1047, C1048, C1049, C1050, C1051, C1052, C1053, C1054, C1055, C1056, C1057, C1059, C1062: 100nF/16V, A_HDJ_Library:C_0402_1005Metric, symbol Device:C
- added C1058: 10uF/10V, A_HDJ_Library:C_0402_1005Metric, symbol Device:C
- added C1060, C1061: 12pF/50V, A_HDJ_Library:C_0402_1005Metric, symbol Device:C
- added J1002: RJ45_RB1-125B8G1A, A_HDJ_Library:RJ45_UDE_RB1-125B8G1A, symbol Connector:RJ45_RB1-125B8G1A
- added R1037, R1038: 10K/1%, A_DFRobot:R_0402, symbol Device:R
- added R1039: 2.49K/1%, A_HDJ_Library:R_0603_1608Metric, symbol Device:R
- added R1040: 1M/1%, A_DFRobot:R_0402, symbol Device:R
- added R1041, R1042: 470R/1%, A_DFRobot:R_0402, symbol Device:R
- added U1007: RTL8111H-CG-RH, A_HDJ_Library:QFN-32-1EP_4x4mm_P0.4mm_EP2.65x2.65mm, symbol [DFR0767]CM4 IoT Router Board Mini(V1.0)-altium-import:root_0_RTL8111H-CG-RH
- added U1013, U1014: ULC0524P, Package_DFN_QFN:Diodes_UDFN-10_1.0x2.5mm_P0.5mm, symbol Power_Protection:D3V3XA4B10LP
- added Y1: 25MHz, A_HDJ_Library:Crystal_SMD_3225-4Pin_3.2x2.5mm, symbol Device:Crystal_GND24
Connections:
- new net: R1037.2, U1007.20 (ISOLATEB)
- new net: R1038.2, U1007.21 (LANWAKEB)
- new net: C1061.2, R1040.2, U1007.28 (CKXTAL1), Y1.1
- new net: C1060.2, R1040.1, U1007.29 (CKXTAL2), Y1.3
- new net: R1039.2, U1007.31 (RSET)
- new net: J1002.L1, R1042.1
- new net: C1062.1, J1002.R1 (CT)
- new net: J1002.L3, R1041.1
- new net +1V0: C1047.2, C1048.2, C1049.2, C1050.2, C1054.2, C1058.2, U1007.22 (DVDD10), U1007.24 (REGOUT), U1007.3 (AVDD10), U1007.30 (AVDD10), U1007.8 (AVDD10)
- new net +3V3: C1051.2, C1055.2, C1059.2, R1037.1, R1038.1, R1041.2, R1042.2, U1007.11 (AVDD33), U1007.23 (VDDREG), U1007.32 (AVDD33)
- new net GND: C1047.1, C1048.1, C1049.1, C1050.1, C1051.1, C1054.1, C1055.1, C1058.1, C1059.1, C1060.1, C1061.1, C1062.2, J1002.R10 (GND), J1002.SH, R1039.1, U1007.33 (GND), U1013.3 (VSS), U1013.8 (VSS), U1014.3 (VSS), U1014.8 (VSS), Y1.2, Y1.4
- new net GbE_PCIe_CLK+: U1007.15 (REFCLK_P)
- new net GbE_PCIe_CLK-: U1007.16 (REFCLK_N)
- new net GbE_PCIe_RX+: C1057.2
- new net GbE_PCIe_RX-: C1053.2
- new net GbE_PCIe_TX+: C1056.2
- new net GbE_PCIe_TX-: C1052.2
- new net HSI+: C1056.1, U1007.13 (HSIP)
- new net HSI-: C1052.1, U1007.14 (HSIN)
- new net HSO+: C1057.1, U1007.17 (HSOP)
- new net HSO-: C1053.1, U1007.18 (HSON)
- new net LED1_1000: J1002.L4, U1007.26 (LED1)
- new net LED2_ACT: J1002.L2, U1007.25 (LED2)
- new net MDI0+: J1002.R2 (TD1+), U1007.1 (MDIP0), U1014.5, U1014.6 (NC)
- new net MDI0-: J1002.R3 (TD1-), U1007.2 (MDIN0), U1014.4, U1014.7 (NC)
- new net MDI1+: J1002.R4 (TD2+), U1007.4 (MDIP1), U1014.2, U1014.9 (NC)
- new net MDI1-: J1002.R5 (TD2-), U1007.5 (MDIN1), U1014.1, U1014.10 (NC)
- new net MDI2+: J1002.R6 (TD3+), U1007.6 (MDIP2), U1013.5, U1013.6 (NC)
- new net MDI2-: J1002.R7 (TD3-), U1007.7 (MDIN2), U1013.4, U1013.7 (NC)
- new net MDI3+: J1002.R8 (TD4+), U1007.9 (MDIP3), U1013.2, U1013.9 (NC)
- new net MDI3-: J1002.R9 (TD4-), U1007.10 (MDIN3), U1013.1, U1013.10 (NC)
- new net ~{CLKREQ4}: U1007.12 (CLKREQB)
- new net ~{PLT_RST}: U1007.19 (PERSTB)
- no-connect marks 0 -> 1
Other:
- note added: "Bob Smith: When designing a metal shell, SH/R10 should connect to shell for better EMC"

Commit message: commit before removing duplicated glasgow
Parts:
- U12: renamed from U1013; footprint Package_DFN_QFN:Diodes_UDFN-10_1.0x2.5mm_P0.5mm -> A_HDJ_Library:Diodes_UDFN-10_1.0x2.5mm_P0.5mm
- U13: renamed from U1014; footprint Package_DFN_QFN:Diodes_UDFN-10_1.0x2.5mm_P0.5mm -> A_HDJ_Library:Diodes_UDFN-10_1.0x2.5mm_P0.5mm
- renumbered C1047 to C65, C1048 to C66, C1049 to C67, C1050 to C68, C1051 to C69, C1052 to C70, C1053 to C71, C1054 to C72, C1055 to C73, C1056 to C74, C1057 to C75, C1058 to C76, C1059 to C77, C1060 to C78, C1061 to C79, C1062 to C80, J1002 to J22, R1037 to R30, R1038 to R31, R1039 to R32, R1040 to R33, R1041 to R34, R1042 to R35, U1007 to U14

Commit message: hdmi-power-finished?
Connections:
- net +3V3 renamed +3V3_highpower
Changed lines of the file:
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@@
 	)
 	(junction
-		(at 261.62 105.41)
-		(diameter 0)
-		(color 0 0 0 0)
-	)
-	(junction
 		(at 97.79 138.43)
 		(diameter 0)
@@
 	)
 	(junction
+		(at 261.62 105.41)
+		(diameter 0)
+		(color 0 0 0 0)
+	)
+	(junction
 		(at 133.35 76.2)
 		(diameter 0)
@@
 	)
 	(symbol
+		(lib_name "+3V3_1")
+		(lib_id "power:+3V3")
+		(at 261.62 105.41 0)
+		(unit 1)
+		(body_style 1)
+		(exclude_from_sim no)
+		(in_bom yes)
+		(on_board yes)
+		(in_pos_files yes)
+		(dnp no)
+		(fields_autoplaced yes)
+		(property "Reference" "#PWR081"
+			(at 261.62 109.22 0)
+			(hide yes)
+			(show_name no)
+			(do_not_autoplace no)
+			(effects
+				(font
+					(size 1.27 1.27)
+				)
+			)
+		)
+		(property "Value" "+3V3_highpower"
+			(at 261.62 100.33 0)
+			(show_name no)
+			(do_not_autoplace no)
+			(effects
+				(font
+					(size 1.27 1.27)
+				)
+			)
+		)
+		(property "Footprint" ""
+			(at 261.62 105.41 0)
+			(hide yes)
+			(show_name no)
+			(do_not_autoplace no)
+			(effects
+				(font
+					(size 1.27 1.27)
+				)
+			)
+		)
+		(property "Datasheet" ""
+			(at 261.62 105.41 0)
+			(hide yes)
+			(show_name no)
+			(do_not_autoplace no)
+			(effects
+				(font
+					(size 1.27 1.27)
+				)
+			)
+		)
+		(property "Description" "Power symbol creates a global label with name \"+3V3\""
+			(at 261.62 105.41 0)
+			(hide yes)
+			(show_name no)
+			(do_not_autoplace no)
+			(effects
+				(font
+					(size 1.27 1.27)
+				)
+			)
+		)
+		(pin "1"
+		)
+		(instances
+			(project "microcyber"
+				(path "/7ac319af-771c-4997-a005-b73a4a9b44ab/3570f5c7-303d-4403-b64c-e6d85fee9a20"
+					(reference "#PWR081")
+					(unit 1)
+				)
+			)
+		)
+	)
+	(symbol
 		(lib_id "Device:C")
 		(at 99.06 77.47 180)
@@
 	)
 	(symbol
-		(lib_id "power:+3V3")
-		(at 119.38 43.18 0)
-		(unit 1)
-		(body_style 1)
-		(exclude_from_sim no)
-		(in_bom yes)
-		(on_board yes)
-		(in_pos_files yes)
-		(dnp no)
-		(fields_autoplaced yes)
-		(property "Reference" "#PWR076"
-			(at 119.38 46.99 0)
-			(hide yes)
-			(show_name no)
-			(do_not_autoplace no)
-			(effects
-				(font
-					(size 1.27 1.27)
-				)
-			)
-		)
-		(property "Value" "+3V3"
-			(at 119.38 38.1 0)
-			(show_name no)
-			(do_not_autoplace no)
-			(effects
-				(font
-					(size 1.27 1.27)
-				)
-			)
-		)
-		(property "Footprint" ""
-			(at 119.38 43.18 0)
-			(hide yes)
-			(show_name no)
-			(do_not_autoplace no)
-			(effects
-				(font
-					(size 1.27 1.27)
-				)
-			)
-		)
-		(property "Datasheet" ""
-			(at 119.38 43.18 0)
-			(hide yes)
-			(show_name no)
-			(do_not_autoplace no)
-			(effects
-				(font
-					(size 1.27 1.27)
-				)
-			)
-		)
-		(property "Description" ""
-			(at 119.38 43.18 0)
-			(hide yes)
-			(show_name no)
-			(do_not_autoplace no)
-			(effects
-				(font
-					(size 1.27 1.27)
-				)
-			)
-		)
-		(pin "1"
-		)
-		(instances
-			(project "microcyber"
-				(path "/7ac319af-771c-4997-a005-b73a4a9b44ab/3570f5c7-303d-4403-b64c-e6d85fee9a20"
-					(reference "#PWR076")
-					(unit 1)
-				)
-			)
-		)
-	)
-	(symbol
 		(lib_id "power:GND")
 		(at 185.42 111.76 0)
@@
 	)
 	(symbol
+		(lib_name "+3V3_1")
+		(lib_id "power:+3V3")
+		(at 113.03 43.18 0)
+		(unit 1)
+		(body_style 1)
+		(exclude_from_sim no)
+		(in_bom yes)
+		(on_board yes)
+		(in_pos_files yes)
+		(dnp no)
+		(fields_autoplaced yes)
+		(property "Reference" "#PWR076"
+			(at 113.03 46.99 0)
+			(hide yes)
+			(show_name no)
+			(do_not_autoplace no)
+			(effects
+				(font
+					(size 1.27 1.27)
+				)
+			)
+		)
+		(property "Value" "+3V3_highpower"
+			(at 113.03 38.1 0)
+			(show_name no)
+			(do_not_autoplace no)
+			(effects
+				(font
+					(size 1.27 1.27)
+				)
+			)
+		)
+		(property "Footprint" ""
+			(at 113.03 43.18 0)
+			(hide yes)
+			(show_name no)
+			(do_not_autoplace no)
+			(effects
+				(font
+					(size 1.27 1.27)
+				)
+			)
+		)
+		(property "Datasheet" ""
+			(at 113.03 43.18 0)
+			(hide yes)
+			(show_name no)
+			(do_not_autoplace no)
+			(effects
+				(font
+					(size 1.27 1.27)
+				)
+			)
+		)
+		(property "Description" "Power symbol creates a global label with name \"+3V3\""
+			(at 113.03 43.18 0)
+			(hide yes)
+			(show_name no)
+			(do_not_autoplace no)
+			(effects
+				(font
+					(size 1.27 1.27)
+				)
+			)
+		)
+		(pin "1"
+		)
+		(instances
+			(project "microcyber"
+				(path "/7ac319af-771c-4997-a005-b73a4a9b44ab/3570f5c7-303d-4403-b64c-e6d85fee9a20"
+					(reference "#PWR076")
+					(unit 1)
+				)
+			)
+		)
+	)
+	(symbol
 		(lib_id "Device:C")
 		(at 106.68 53.34 180)
@@
 					(unit 1)
 				)
-			)
-		)
-	)
-	(symbol
-		(lib_id "power:+3V3")
-		(at 261.62 105.41 0)
-		(unit 1)
-		(body_style 1)
-		(exclude_from_sim no)
-		(in_bom yes)
-		(on_board yes)
-		(in_pos_files yes)
-		(dnp no)
-		(fields_autoplaced yes)
-		(property "Reference" "#PWR081"
-			(at 261.62 109.22 0)
-			(hide yes)
-			(show_name no)
-			(do_not_autoplace no)
-			(effects
-				(font
-					(size 1.27 1.27)
-				)
-			)
-		)
-		(property "Value" "+3V3"
-			(at 261.62 100.33 0)
-			(show_name no)
-			(do_not_autoplace no)
-			(effects
-				(font
-					(size 1.27 1.27)
-				)
-			)
-		)
-		(property "Footprint" ""
-			(at 261.62 105.41 0)
-			(hide yes)
-			(show_name no)
-			(do_not_autoplace no)
-			(effects
-				(font
-					(size 1.27 1.27)
-				)
-			)
-		)
-		(property "Datasheet" ""
-			(at 261.62 105.41 0)
-			(hide yes)
-			(show_name no)
-			(do_not_autoplace no)
-			(effects
-				(font
-					(size 1.27 1.27)
-				)
-			)
-		)
-		(property "Description" ""
-			(at 261.62 105.41 0)
-			(hide yes)
-			(show_name no)
-			(do_not_autoplace no)
-			(effects
-				(font
-					(size 1.27 1.27)
-				)
-			)
-		)
-		(pin "1"
-		)
-		(instances
-			(project "microcyber"
-				(path "/7ac319af-771c-4997-a005-b73a4a9b44ab/3570f5c7-303d-4403-b64c-e6d85fee9a20"
-					(reference "#PWR081")
-					(unit 1)
-				)

Commit message: V4 done ???
Parts:
- U12, U13: now fitted; now in the parts list
Changed lines of the file:
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@@
 		(body_style 1)
 		(exclude_from_sim no)
-		(in_bom no)
+		(in_bom yes)
 		(on_board yes)
 		(in_pos_files yes)
-		(dnp yes)
+		(dnp no)
 		(property "Reference" "U12"
 			(at 115.57 156.21 0)
@@
 		(body_style 1)
 		(exclude_from_sim no)
-		(in_bom no)
+		(in_bom yes)
 		(on_board yes)
 		(in_pos_files yes)
-		(dnp yes)
+		(dnp no)
 		(property "Reference" "U13"
 			(at 115.57 182.88 0)

Commit message: last push before editing with the grid view (gonna break everything)
Parts:
- C65, C66, C67, C68, C69, C70, C71, C72, C73, C74, C75, C77, C80: value 100nF/16V -> 100n; MPN (none) -> 0402B104K160NT
- C76: value 10uF/10V -> 10u; MPN (none) -> CC0402MRX5R6BB106
- C78, C79: value 12pF/50V -> 12p; MPN (none) -> CC0402JRNPO9BN120
- J22: MPN (none) -> RB1-125B8G1A
- R30, R31: value 10K/1% -> 10K; MPN (none) -> C2889342
- R32: value 2.49K/1% -> 2K49; DF_Comment 贴片电阻0603-2.49K-1%(0603-1.6*0.8*0.4) -> (none); MPN (none) -> RK73H1JLTD2491F
- R33: value 1M/1% -> 1M; DF_Comment 贴片电阻0402-1M-1% -> (none); MPN (none) -> CC0402KRX7R9BB104
- R34, R35: value 470R/1% -> 470; DF_Comment 贴片电阻0402-470R-1% -> (none); MPN (none) -> ERJ-2RKF4700X
- U12, U13: MPN (none) -> ULC0524P
- U14: MPN (none) -> RTL8111H-CG-RH
- Y1: MPN (none) -> C9900024673

Commit message: added MPN to all parts by hand :'(
Parts:
- C65, C66, C67, C68, C69, C70, C71, C72, C73, C74, C75, C77, C80: value 100n -> u1; MPN 0402B104K160NT -> C1005X7R1H104K050BE
- C76: footprint A_HDJ_Library:C_0402_1005Metric -> A_DFRobot:C_0603; DF_Comment 贴片电容0402-10UF-10V-X5R_GRM155R61A106ME44D -> (none); MPN CC0402MRX5R6BB106 -> GRM188R61E106KA73D; SCH_Show_Footprint C0402 -> (none)
- R30, R31: MPN C2889342 -> RCS040210K0FKED
Changed lines of the file:
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@@
 			)
 		)
-		(property "Value" "100n"
+		(property "Value" "u1"
 			(at 113.03 101.6 90)
 			(show_name no)
@@
 			)
 		)
-		(property "MPN" "0402B104K160NT"
+		(property "MPN" "C1005X7R1H104K050BE"
 			(at 106.68 102.87 0)
 			(hide yes)
@@
 			)
 		)
-		(property "Value" "100n"
+		(property "Value" "u1"
 			(at 93.98 83.82 90)
 			(show_name no)
@@
 			)
 		)
-		(property "MPN" "0402B104K160NT"
+		(property "MPN" "C1005X7R1H104K050BE"
 			(at 92.71 77.47 0)
 			(hide yes)
@@
 			)
 		)
-		(property "Value" "100n"
+		(property "Value" "u1"
 			(at 87.63 83.82 90)
 			(show_name no)
@@
 			)
 		)
-		(property "MPN" "0402B104K160NT"
+		(property "MPN" "C1005X7R1H104K050BE"
 			(at 86.36 77.47 0)
 			(hide yes)
@@
 			)
 		)
-		(property "Value" "100n"
+		(property "Value" "u1"
 			(at 113.03 93.98 90)
 			(show_name no)
@@
 			)
 		)
-		(property "MPN" "0402B104K160NT"
+		(property "MPN" "C1005X7R1H104K050BE"
 			(at 106.68 95.25 0)
 			(hide yes)
@@
 			)
 		)
-		(property "Value" "100n"
+		(property "Value" "u1"
 			(at 106.68 83.82 90)
 			(show_name no)
@@
 			)
 		)
-		(property "MPN" "0402B104K160NT"
+		(property "MPN" "C1005X7R1H104K050BE"
 			(at 105.41 77.47 0)
 			(hide yes)
@@
 			)
 		)
-		(property "MPN" "C2889342"
+		(property "MPN" "RCS040210K0FKED"
 			(at 129.54 53.34 0)
 			(hide yes)
@@
 			)
 		)
-		(property "Value" "100n"
+		(property "Value" "u1"
 			(at 100.33 83.82 90)
 			(show_name no)
@@
 			)
 		)
-		(property "MPN" "0402B104K160NT"
+		(property "MPN" "C1005X7R1H104K050BE"
 			(at 99.06 77.47 0)
 			(hide yes)
@@
 			)
 		)
-		(property "Value" "100n"
+		(property "Value" "u1"
 			(at 81.28 83.82 90)
 			(show_name no)
@@
 			)
 		)
-		(property "MPN" "0402B104K160NT"
+		(property "MPN" "C1005X7R1H104K050BE"
 			(at 80.01 77.47 0)
 			(hide yes)
@@
 			)
 		)
-		(property "Value" "100n"
+		(property "Value" "u1"
 			(at 114.3 59.69 90)
 			(show_name no)
@@
 			)
 		)
-		(property "MPN" "0402B104K160NT"
+		(property "MPN" "C1005X7R1H104K050BE"
 			(at 113.03 53.34 90)
 			(hide yes)
@@
 			)
 		)
-		(property "Value" "100n"
+		(property "Value" "u1"
 			(at 101.6 59.69 90)
 			(show_name no)
@@
 			)
 		)
-		(property "MPN" "0402B104K160NT"
+		(property "MPN" "C1005X7R1H104K050BE"
 			(at 100.33 53.34 90)
 			(hide yes)
@@
 			)
 		)
-		(property "Value" "100n"
+		(property "Value" "u1"
 			(at 220.98 91.44 90)
 			(show_name no)
@@
 			)
 		)
-		(property "MPN" "0402B104K160NT"
+		(property "MPN" "C1005X7R1H104K050BE"
 			(at 215.9 92.71 0)
 			(hide yes)
@@
 			)
 		)
-		(property "Value" "100n"
+		(property "Value" "u1"
 			(at 106.68 91.44 90)
 			(show_name no)
@@
 			)
 		)
-		(property "MPN" "0402B104K160NT"
+		(property "MPN" "C1005X7R1H104K050BE"
 			(at 100.33 92.71 0)
 			(hide yes)
@@
 			)
 		)
-		(property "Value" "100n"
+		(property "Value" "u1"
 			(at 106.68 99.06 90)
 			(show_name no)
@@
 			)
 		)
-		(property "MPN" "0402B104K160NT"
+		(property "MPN" "C1005X7R1H104K050BE"
 			(at 100.33 100.33 0)
 			(hide yes)
@@
 			)
 		)
-		(property "MPN" "C2889342"
+		(property "MPN" "RCS040210K0FKED"
 			(at 119.38 53.34 0)
 			(hide yes)
@@
 			)
 		)
-		(property "Value" "100n"
+		(property "Value" "u1"
 			(at 107.95 59.69 90)
 			(show_name no)
@@
 			)
 		)
-		(property "MPN" "0402B104K160NT"
+		(property "MPN" "C1005X7R1H104K050BE"
 			(at 106.68 53.34 90)
 			(hide yes)
@@
 			)
 		)
-		(property "Footprint" "A_HDJ_Library:C_0402_1005Metric"
+		(property "Footprint" "A_DFRobot:C_0603"
 			(at 110.7948 73.66 0)
 			(hide yes)
@@
 			)
 		)
-		(property "DF_Comment" "贴片电容0402-10UF-10V-X5R_GRM155R61A106ME44D"
+		(property "DF_Comment" ""
 			(at 111.76 77.47 0)
 			(hide yes)
@@
 			)
 		)
-		(property "SCH_Show_Footprint" "C0402"
+		(property "SCH_Show_Footprint" ""
 			(at 111.76 77.47 0)
 			(hide yes)
@@
 			)
 		)
-		(property "MPN" "  CC0402MRX5R6BB106"
+		(property "MPN" "GRM188R61E106KA73D"
 			(at 111.76 77.47 0)
 			(hide yes)
