File: M2_MKEY.kicad_sch (KiCad schematic)
At the start: 15 parts, among them J24 Bus_M.2_Socket_M

Commit message: added MPN to all parts by hand :'(
Parts:
- C90: footprint A_HDJ_Library:C_0402_1005Metric -> A_DFRobot:C_0603; MPN MLASL168BB5106MTNB33 -> GRM188R61E106KA73D
- C91, C93: MPN C0402C104J4RECAUTO -> C1005X7R1H104K050BE
- C92: footprint A_HDJ_Library:C_0402_1005Metric -> A_DFRobot:C_0603; MPN MLASL168BB5106MTNB33 -> GRM188R61E106KA73D; SCH_Show_Footprint C0402 -> (none)
- R39: MPN C2889341 -> MCS0402HZ0000ZE100
- R40: MPN 560112110087 -> RCS04022K20FKED
Changed lines of the file:
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@@
 			)
 		)
-		(property "MPN" "C0402C104J4RECAUTO"
+		(property "MPN" "C1005X7R1H104K050BE"
 			(at 134.62 33.02 0)
 			(hide yes)
@@
 			)
 		)
-		(property "MPN" "560112110087"
+		(property "MPN" "RCS04022K20FKED"
 			(at 166.37 99.06 0)
 			(hide yes)
@@
 			)
 		)
-		(property "Footprint" "A_HDJ_Library:C_0402_1005Metric"
+		(property "Footprint" "A_DFRobot:C_0603"
 			(at 130.81 40.3352 0)
 			(hide yes)
@@
 			)
 		)
-		(property "SCH_Show_Footprint" "C0402"
+		(property "SCH_Show_Footprint" ""
 			(at 134.62 39.37 0)
 			(hide yes)
@@
 			)
 		)
-		(property "MPN" "MLASL168BB5106MTNB33"
+		(property "MPN" "GRM188R61E106KA73D"
 			(at 134.62 39.37 0)
 			(hide yes)
@@
 			)
 		)
-		(property "MPN" "C0402C104J4RECAUTO"
+		(property "MPN" "C1005X7R1H104K050BE"
 			(at 134.62 45.72 0)
 			(hide yes)
@@
 			)
 		)
-		(property "Footprint" "A_HDJ_Library:C_0402_1005Metric"
+		(property "Footprint" "A_DFRobot:C_0603"
 			(at 130.81 27.6352 0)
 			(hide yes)
@@
 			)
 		)
-		(property "MPN" "MLASL168BB5106MTNB33"
+		(property "MPN" "GRM188R61E106KA73D"
 			(at 134.62 26.67 0)
 			(hide yes)
@@
 			)
 		)
-		(property "MPN" "C2889341"
+		(property "MPN" "MCS0402HZ0000ZE100"
 			(at 163.83 128.27 0)
 			(hide yes)
