File: microcyber.kicad_pcb (KiCad board)
At the start: 6 copper layers, 190.8 x 134 mm, 497 parts, among them J1 Conn_01x03_Pin, J2 Bus_M.2_Socket_E, J22 RJ45_RB1-125B8G1A, J24 Bus_M.2_Socket_M, J25 AUX, J26 Conn_01x02, J27 PinHeader_2x22_P1.27mm, J28 IDC-Header_2x10_P2.54mm, J29 Conn_01x08, J30 Conn_01x08, J31 Bus_M.2_Socket_E, J32 HDMI_D_1.4, J34 Bus_M.2_Socket_E, J5 Conn_01x01_Socket, J501 USB_C_Receptacle, J6 Conn_01x01_Socket, J7 USB3_A, J8 Conn_01x02_Socket, P1 1775862-2, Q11 2N7002, Q12 2SK3018, Q13 2SK3018, Q14 2SK3018, Q401 2N7002, SW1 RST, SW401 SW_Push, SW402 SW_Push, U1 ADV7623BSTZ, U12 ULC0524P, U13 ULC0524P, U14 RTL8111H-CG-RH, U15 ULC0524P, U16 ULC0524P, U18 TPD3S014, U19 CY7C68013A-56LTX, U2 NC7SZ125M5, U20 CAT24M01X, U21 BL24C256A-SFRC, U22 ICE40HX8K-BG121, U23 APX811-40UG-7, U24 TLV75533PDRVR, U25 TLV73312PQDRVR, U26 SN74LVC1T45DCKR, U27 SN74LVC1T45DCKR, U28 SN74LVC1T45DCKR, U29 SN74LVC1T45DCKR, U3 TPPM0110DWPR, U30 SN74LVC1T45DCKR, U31 SN74LVC1T45DCKR, U32 SN74LVC1T45DCKR, U33 SN74LVC1T45DCKR, U34 SN74LVC1T45DCKR, U35 PCA6408APW, U36 TPS73101DBV, U37 DAC081C081CIMK, U38 INA233, U4 TPS548A23VANR, U403 AP63200WU, U43 TPAZ1023-04F, U44 TPAZ1023-04F, U501 ULC0524P, U503 ULC0524P, U506 LM73100RPWR, U507 AT25DN512C-MAHF-T, U508 TPS65988DHRSHR, Y1 25MHz, Y2 24M, Y3 ABM8G-28.63636MHZ-18-D2Y-T

Commit message: resend fab
Routing:
- net GND: track 323.8 -> 325.4 mm, vias 841 -> 840
