File: edgeboard/edgeboard/edgeboard.kicad_sch (KiCad schematic)
At the start: 0 parts

Commit message: added USB-C
Parts:
- added BT1, BT2: BK-18650-PC6, keyswitch:BAT_BK-18650-PC6, symbol BK-18650-PC6:BK-18650-PC6
- added BT601, BT602, BT603: 1043P, ComputemanParts:BAT_1042P, symbol 1043p:1043P
- added C501, C502, C524, C526, C527, C532, C533: 100nF/50V, A_HDJ_Library:C_0402_1005Metric, symbol Device:C
- added C503, C504, C505, C506: 47pF, A_HDJ_Library:C_0402_1005Metric, symbol Device:C
- added C507, C508, C509, C510, C515, C516, C517, C518: 330n, A_HDJ_Library:C_0402_1005Metric, symbol Device:C
- added C511, C512, C513, C514, C519, C520, C521, C522: 220n, A_HDJ_Library:C_0402_1005Metric, symbol Device:C
- added C523: 22uF/10V, A_HDJ_Library:C_0603_1608Metric, symbol Device:C
- added C525, C531: 10uF/10V, A_HDJ_Library:C_0603_1608Metric, symbol Device:C
- added C528: 4.7uF/10V, A_HDJ_Library:C_0402_1005Metric, symbol Device:C
- added C529, C530, C534, C535: 47pF/50V, A_HDJ_Library:C_0402_1005Metric, symbol Device:C
- added C601, C602, C613, C614, C615, C618, C623: 0.1u, A_HDJ_Library:C_0402_1005Metric, symbol Device:C
- added C603: 3x10uF MLCC, A_HDJ_Library:C_0402_1005Metric, symbol Device:C
- added C604, C605: 47n, A_HDJ_Library:C_0402_1005Metric, symbol Device:C
- added C606, C607, C608, C609: 10uF MLCC, A_HDJ_Library:C_0402_1005Metric, symbol Device:C
- added C610, C611: 33n, A_HDJ_Library:C_0402_1005Metric, symbol Device:C
- added C612: 0.47u, A_HDJ_Library:C_0402_1005Metric, symbol Device:C
- added C616: 33p, A_HDJ_Library:C_0402_1005Metric, symbol Device:C
- added C617: 1800p, A_HDJ_Library:C_0402_1005Metric, symbol Device:C
- added C619: 1u, A_HDJ_Library:C_0402_1005Metric, symbol Device:C
- added C620, C625: 2.2u, A_HDJ_Library:C_0402_1005Metric, symbol Device:C
- added C621: 15p, A_HDJ_Library:C_0402_1005Metric, symbol Device:C
- added C622: 680p, A_HDJ_Library:C_0402_1005Metric, symbol Device:C
- added C624: 100p, A_HDJ_Library:C_0402_1005Metric, symbol Device:C
- added D501, D502, D503, D504, D505, D506, D507, D508, D509, D510, D511, D512: ESD5V0B03, A_HDJ_Library:D_0402_1005Metric, symbol Diode:ESD9B5.0ST5G
- added D515, D516, D517, D518, D519, D520, D521, D522, D523, D524, D525: ESD9B3.3ST5GOSCT-ND, A_HDJ_Library:D_0402_1005Metric, symbol Diode:ESD9B5.0ST5G
- added D601: BAT54HT1, A_HDJ_Library:D_SOD-323, symbol Device:D_Schottky
- added J1: Bus_PCI_Express_Mini, mpcie:mpcie-full-card, symbol Connector:Bus_PCI_Express_Mini
- added J501, J502: USB_C_Receptacle, Connector_USB:USB_C_Receptacle_Amphenol_12401610E4-2A, symbol Connector:USB_C_Receptacle
- added J601: JST XH 4 pin, Connector_JST:JST_XH_S4B-XH-A_1x04_P2.50mm_Horizontal, symbol Connector:Conn_01x04_Socket
- added JP601: Jumper_2_Bridged, Jumper:SolderJumper-2_P1.3mm_Bridged_Pad1.0x1.5mm, symbol Jumper:Jumper_2_Bridged
- added L601: 2.2uH 4.5A+, Inductor_SMD:L_Bourns_SRP5030T, symbol Device:L
- added Q601, Q602, Q603, Q604, Q605, Q606: CSD17551Q3A, Package_SO:Vishay_PowerPAK_1212-8_Single, symbol Transistor_FET:Si7336ADP
- added Q607: CSD25402Q3A, Package_SO:Vishay_PowerPAK_1212-8_Single, symbol Simulation_SPICE:PMOS
- added R501, R502, R503, R504, R508, R509, R510, R511, R512: 100K/1%, A_HDJ_Library:R_0402_1005Metric, symbol Device:R
- added R505, R506: 10K/1%, A_HDJ_Library:R_0402_1005Metric, symbol Device:R
- added R507: 100K, A_HDJ_Library:R_0402_1005Metric, symbol Device:R
- added R513, R612, R619: 10K, A_HDJ_Library:R_0402_1005Metric, symbol Device:R
- added R514: 19.1K/1%, A_HDJ_Library:R_0402_1005Metric, symbol Device:R
- added R601, R613: 10m, A_HDJ_Library:R_0805_2012Metric, symbol Device:R
- added R602, R603: 10M, A_HDJ_Library:R_0402_1005Metric, symbol Device:R
- added R604, R605: 4.99, A_HDJ_Library:R_0402_1005Metric, symbol Device:R
- added R606, R607: 5.1k, A_HDJ_Library:R_0402_1005Metric, symbol Device:R
- added R608, R610, R615, R618, R621, R624: 100, A_HDJ_Library:R_0402_1005Metric, symbol Device:R
- added R609: 1, A_HDJ_Library:R_0402_1005Metric, symbol Device:R
- added R611, R614, R617: 10, A_HDJ_Library:R_0402_1005Metric, symbol Device:R
- added R616: 40.2k, A_HDJ_Library:R_0402_1005Metric, symbol Device:R
- added R620: 10k, A_HDJ_Library:R_0402_1005Metric, symbol Device:R
- added R622, R625, R626, R628: TBD, A_HDJ_Library:R_0402_1005Metric, symbol Device:R
- added R623: 0.001, A_HDJ_Library:R_0805_2012Metric, symbol Device:R
- added R627: 137K, A_HDJ_Library:R_0402_1005Metric, symbol Device:R
- added SW1, SW2, SW3, SW4: SW_Push, PCM_Switch_Keyboard_Kailh:SW_Kailh_Choc_Mini_1.25u_90deg, symbol Switch:SW_Push
- added SW10: SW_Push, PCM_Switch_Keyboard_Kailh:SW_Kailh_Choc_Mini_ISOEnter_180deg, symbol Switch:SW_Push
- added SW11, SW12, SW13, SW14, SW15, SW16, SW17, SW18, SW19, SW20, SW21, SW22, SW23, SW6, SW7, SW8: SW_Push, PCM_Switch_Keyboard_Kailh:SW_Kailh_Choc_Mini_1.00u, symbol Switch:SW_Push
- added SW5: SW_Push, PCM_Switch_Keyboard_Kailh:SW_Kailh_Choc_Mini_1.50u, symbol Switch:SW_Push
- added SW9: SW_Push, PCM_Switch_Keyboard_Kailh:SW_Kailh_Choc_Mini_1.50u_90deg, symbol Switch:SW_Push
- added TH601: BN35-3H103, Connector_PinHeader_2.54mm:PinHeader_1x02_P2.54mm_Vertical, symbol Device:Thermistor_NTC
- added TP601: VBAT, TestPoint:TestPoint_Pad_D1.5mm, symbol Connector:TestPoint
- added TP602: VCHARGE, TestPoint:TestPoint_Pad_D1.5mm, symbol Connector:TestPoint
- added TP603: VSYSTEM, TestPoint:TestPoint_Pad_D1.5mm, symbol Connector:TestPoint
- added TP604: PSYS, TestPoint:TestPoint_Pad_D1.5mm, symbol Connector:TestPoint
- added TP605: PROCHOT, TestPoint:TestPoint_Pad_D1.5mm, symbol Connector:TestPoint
- added TP606: IBAT, TestPoint:TestPoint_Pad_D1.5mm, symbol Connector:TestPoint
- added TP607: CHRG_OK, TestPoint:TestPoint_Pad_D1.5mm, symbol Connector:TestPoint
- added U501, U502, U503, U504, U509, U510, U511: ULC0524P, A_HDJ_Library:Diodes_UDFN-10_1.0x2.5mm_P0.5mm, symbol Power_Protection:D3V3XA4B10LP
- added U505, U506: LM73100RPWR, ComputemanParts:IC_LM73100RPWR, symbol lm73100:LM73100RPWR
- added U507: AT25DN512C-MAHF-T, Package_DFN_QFN:DFN-8-1EP_3x2mm_P0.5mm_EP1.75x1.45mm, symbol Memory_EEPROM:AT25xxx-MA
- added U508: TPS65988DHRSHR, ComputemanParts:IC_TPS65987DDHRSHR, symbol tps65988:TPS65988DHRSHR
- added U601: BQ25710RSNT, ComputemanParts:QFN40P400X400X80-33N, symbol bq25710:BQ25710RSNT
- added U602: BQ40Z50RSMR-R2, ComputemanParts:QFN40P400X400X100-33N, symbol bq40z50:BQ40Z50RSMR-R2
Connections:
- new net: U509.5, U509.6 (NC)
- new net: C619.1, R617.1, R622.1, R626.1, U601.7 (VDDA)
- new net: R622.2, R625.1, U601.18 (CELL_BATPRESZ)
- new net: Q601.4 (G), R602.2, R606.1
- new net: Q601.5 (D), Q602.5 (D), R608.1
- new net: C601.2, C602.1
- new net: R513.2, U508.44 (HRESET)
- new net: BT601.N, BT602.P, J601.2 (Pin_2), R615.1
- new net: BT602.N, BT603.P, J601.3 (Pin_3), R618.1
- new net: C523.2, U508.35 (LDO_1V8)
- new net: R606.2, U602.31 (CHG)
- new net: C621.1, R620.1, U601.17 (COMP2)
- new net: C622.1, R620.2
- new net: U507.1 (~{CS}), U508.39 (~{SPI_CS})
- new net: U507.2 (MISO), U508.36 (SPI_POCI)
- new net: U507.5 (MOSI), U508.37 (SPI_PICO)
- new net: U507.6 (SCK), U508.38 (SPI_CLK)
- new net: C620.1, R617.2, U601.28 (REGN)
- new net: C612.1, R609.2, U601.1 (VBUS)
- new net: C625.1, U602.1 (PBI)
- new net: C614.1, C615.2, R615.2, U602.4 (VC2)
- new net: C614.2, R610.2, U602.2 (VC4), U602.3 (VC3)
- new net: C617.1, R616.2
- new net: Q602.4 (G), R603.2, R607.1
- new net: R607.2, U602.28 (DSG)
- new net: C605.1, L601.2, Q604.1 (S), Q604.2 (S), Q604.3 (S), Q606.5 (D), U601.23 (SW2)
- new net: C605.2, U601.25 (BTST2)
- new net: R612.2, U602.27 (PACK)
- new net: JP601.2 (B), TH601.2, U602.10 (TS1)
- new net: TP606.1, U601.9 (IBAT)
- new net: C604.1, L601.1, Q603.1 (S), Q603.2 (S), Q603.3 (S), Q605.5 (D), U601.32 (SW1)
- new net: TP607.1, U601.4 (CHRG_OK)
- new net: Q604.4 (G), U601.24 (HIDRV2)
- new net: R512.2, R514.1, U508.6 (ADCIN1)
- new net: C616.1, R616.1, U601.16 (COMP1)
- new net: C615.1, C618.2, R618.2, U602.5 (VC1)
- new net: R619.2, U602.16 (~{PRES}/~{SHUTDN})
- new net: R608.2, U602.26 (VCC)
- new net: D601.1 (K), U602.32 (BAT)
- new net: R624.2, U602.6 (SRN)
- new net: R621.2, U602.8 (SRP)
- new net: C624.1, R627.1, U601.8 (IADPT)
- new net: C611.1, R605.2, U601.2 (ACN)
- new net: Q607.4 (G), U601.21 (~{BATDRV})
- new net: R611.2, U601.20 (SRP)
- new net: U508.15 (DRAIN1__1), U508.19 (DRAIN1__2), U508.58 (DRAIN1__3), U508.58_1 (DRAIN1_PAD), U508.58_2 (DRAIN1_PAD), U508.58_3 (DRAIN1_PAD), U508.58_4 (DRAIN1_PAD), U508.58_5 (DRAIN1_PAD), U508.58_6 (DRAIN1_PAD), U508.8 (DRAIN1)
- new net: R507.2, U508.17 (GPIO1)
- new net: R505.1, U508.27 (I2C1_SCL)
- new net: R506.1, U508.28 (I2C1_SDA)
- new net: U508.52 (DRAIN2__1), U508.56 (DRAIN2__2), U508.57 (DRAIN2__3), U508.57_1 (DRAIN2_PAD), U508.57_2 (DRAIN2_PAD), U508.57_3 (DRAIN2_PAD), U508.57_4 (DRAIN2_PAD), U508.57_5 (DRAIN2_PAD), U508.57_6 (DRAIN2_PAD), U508.7 (DRAIN2)
- new net: Q606.4 (G), U601.26 (LODRV2)
- new net: Q605.4 (G), U601.29 (LODRV1)
- new net: TP604.1, U601.10 (PSYS)
- new net: TP605.1, U601.11 (~{PROCHOT})
- new net: R614.2, U601.19 (SRN)
- new net: C610.1, R604.2, U601.3 (ACP)
- new net: C604.2, U601.30 (BTST1)
- new net: Q603.4 (G), U601.31 (HIDRV1)
- new net: R626.2, R628.1, U601.6 (ILIM_HIZ)
- new net: Q603.5 (D), R601.2, R605.1
- new net: J1.15 (GND), J1.18 (GND), J1.21 (GND), J1.26 (GND), J1.27 (GND), J1.29 (GND), J1.34 (GND), J1.35 (GND), J1.37 (GND), J1.4 (GND), J1.40 (GND), J1.43 (GND), J1.50 (GND), J1.9 (GND)
- new net +3V3: C531.2, U508.5 (VIN_3V3)
- new net +3V3_TPS: C525.2, C527.2, R505.2, R506.2, R512.1, U507.8 (VCC), U508.9 (LDO_3V3)
- new net +5V: C528.2, U508.25 (PP1_CABLE), U508.46 (PP2_CABLE)
- new net -BATT: BT603.N, C623.1, J601.4 (Pin_4), R621.1, R623.1
- new net BTP_INT: U602.15 (BTP_INT)
- new net DISP1_HPD: R510.1, U508.30 (GPIO3(HPD1))
- new net DISP2_HPD: R511.1, U508.31 (GPIO4(HPD2))
- new net EXT_VBUS_SOURCE1: R501.2, U506.1 (EN/UVLO), U508.48 (GPIO16(PP_EXT1))
- new net EXT_VBUS_SOURCE2: R502.2, U505.1 (EN/UVLO), U508.49 (GPIO17(PP_EXT2))
- new net GND: C501.2, C502.2, C503.2, C504.2, C505.2, C506.2, C523.1, C525.1, C527.1, C528.1, C529.2, C530.2, C531.1, C534.2, C535.2, C603.2, C606.2, C607.2, C608.2, C609.2, C610.2, C611.2, C612.2, C616.2, C617.2, C618.1, C619.2, C620.2, C621.2, C622.2, C623.2, C624.2, C625.2, D501.1 (A1), D502.1 (A1), D503.1 (A1), D504.1 (A1), D505.1 (A1), D506.1 (A1), D507.1 (A1), D508.1 (A1), D509.1 (A1), D510.1 (A1), D511.1 (A1), D512.1 (A1), D515.1 (A1), D516.1 (A1), D517.1 (A1), D518.1 (A1), D519.1 (A1), D520.1 (A1), D521.1 (A1), D522.1 (A1), D523.1 (A1), D524.1 (A1), D525.1 (A1), J501.A1 (GND), J501.A12 (GND), J501.B1 (GND), J501.B12 (GND), J501.S1 (SHIELD), J502.A1 (GND), J502.A12 (GND), J502.B1 (GND), J502.B12 (GND), J502.S1 (SHIELD), JP601.1 (A), Q605.1 (S), Q605.2 (S), Q605.3 (S), Q606.1 (S), Q606.2 (S), Q606.3 (S), R501.1, R502.1, R507.1, R510.2, R511.2, R513.1, R514.2, R619.1, R623.2, R624.1, R625.2, R627.2, R628.2, TH601.1, U501.3 (VSS), U501.8 (VSS), U502.3 (VSS), U502.8 (VSS), U503.3 (VSS), U503.8 (VSS), U504.3 (VSS), U504.8 (VSS), U505.2 (OVLO), U505.4 (PGTH), U505.8 (GND), U505.9 (IMON), U506.2 (OVLO), U506.4 (PGTH), U506.8 (GND), U506.9 (IMON), U507.4 (GND), U507.9 (GND), U508.10 (ADCIN2), U508.20 (GND), U508.51 (GND__1), U508.59 (THERMALPAD(PPAD)), U508.59_1 (THERMALPAD(PPAD)), U508.59_10 (THERMALPAD(PPAD)), U508.59_11 (THERMALPAD(PPAD)), U508.59_2 (THERMALPAD(PPAD)), U508.59_3 (THERMALPAD(PPAD)), U508.59_4 (THERMALPAD(PPAD)), U508.59_5 (THERMALPAD(PPAD)), U508.59_6 (THERMALPAD(PPAD)), U508.59_7 (THERMALPAD(PPAD)), U508.59_8 (THERMALPAD(PPAD)), U508.59_9 (THERMALPAD(PPAD)), U509.3 (VSS), U509.8 (VSS), U510.3 (VSS), U510.8 (VSS), U511.3 (VSS), U511.8 (VSS), U601.14 (CMPIN), U601.27 (PGND), U601.5 (OTG/VAP), U602.11 (TS2), U602.12 (TS3), U602.13 (TS4), U602.17 (~{DISP}), U602.23 (PTC), U602.24 (PTCEN), U602.33 (EXP), U602.33_1 (EXP__1), U602.9 (VSS)
- new net GPIO_1: D517.2 (A2), U511.1, U511.10 (NC)
- new net GPIO_2: D516.2 (A2), U511.4, U511.7 (NC)
- new net GPIO_3: D515.2 (A2), U511.2, U511.9 (NC)
- new net GPIO_4: D518.2 (A2), U511.5, U511.6 (NC)
- new net GPIO_5: D519.2 (A2), U510.1, U510.10 (NC)
- new net GPIO_6: D520.2 (A2), U510.4, U510.7 (NC)
- new net GPIO_7: D521.2 (A2), U510.2, U510.9 (NC)
- new net GPIO_8: D522.2 (A2), U510.5, U510.6 (NC)
- new net PACK+: BT601.P, C601.1, D601.2 (A), J601.1 (Pin_1), Q601.1 (S), Q601.2 (S), Q601.3 (S), R602.1, R610.1
- new net SMB_ALERT: D525.2 (A2), U509.4, U509.7 (NC)
- new net SMB_CLK: D524.2 (A2), U509.2, U509.9 (NC), U601.13 (SCL), U602.19 (SMBC)
- new net SMB_DATA: D523.2 (A2), U509.1, U509.10 (NC), U601.12 (SDA), U602.18 (SMBD)
- new net SMLCLK: U508.32 (I2C2_SCL)
- new net SMLDAT: U508.33 (I2C2_SDA)
- new net USBC1_AUX+: C524.1
- new net USBC1_AUX-: C526.1
- new net USBC1_CC1: C504.1, D501.2 (A2), J501.A5 (CC1), U508.24 (C1_CC1)
- new net USBC1_CC2: C503.1, D502.2 (A2), J501.B5 (CC2), U508.26 (C1_CC2)
- new net USBC1_CONN_RX1+: C509.1, J501.B11 (RX1+)
- new net USBC1_CONN_RX1-: C507.1, J501.B10 (RX1-)
- new net USBC1_CONN_RX2+: C517.1, J501.A11 (RX2+)
- new net USBC1_CONN_RX2-: C515.1, J501.A10 (RX2-)
- new net USBC1_CONN_TX1+: C513.1, J501.A2 (TX1+)
- new net USBC1_CONN_TX1-: C511.1, J501.A3 (TX1-)
- new net USBC1_CONN_TX2+: C521.1, J501.B2 (TX2+)
- new net USBC1_CONN_TX2-: C519.1, J501.B3 (TX2-)
- new net USBC1_DDCCLK: R503.1
- new net USBC1_DDCDAT: R504.1
- new net USBC1_SBU1: C524.2, C529.1, D505.2 (A2), J501.A8 (SBU1), R504.2
- new net USBC1_SBU2: C526.2, C530.1, D506.2 (A2), J501.B8 (SBU2), R503.2
- new net USBC1_TX0_D+: C513.2, U501.4, U501.7 (NC)
- new net USBC1_TX0_D-: C511.2, U501.5, U501.6 (NC)
- new net USBC1_TX1_D+: C521.2, U503.5, U503.6 (NC)
- new net USBC1_TX1_D-: C519.2, U503.4, U503.7 (NC)
- new net USBC1_TXRX0_D+: C509.2, U501.1, U501.10 (NC)
- new net USBC1_TXRX0_D-: C507.2, U501.2, U501.9 (NC)
- new net USBC1_TXRX1_D+: C517.2, U503.2, U503.9 (NC)
- new net USBC1_TXRX1_D-: C515.2, U503.1, U503.10 (NC)
- new net USBC1_USB2_D+: D503.2 (A2), J501.A6 (D+), J501.B6 (D+)
- new net USBC1_USB2_D-: D504.2 (A2), J501.A7 (D-), J501.B7 (D-)
- new net USBC1_VBUS: C501.1, J501.A4 (VBUS), J501.A9 (VBUS), J501.B4 (VBUS), J501.B9 (VBUS), U506.6 (OUT), U508.13 (VBUS1)
- new net USBC2_AUX+: C532.1
- new net USBC2_AUX-: C533.1
- new net USBC2_CC1: C506.1, D507.2 (A2), J502.A5 (CC1), U508.45 (C2_CC1)
- new net USBC2_CC2: C505.1, D508.2 (A2), J502.B5 (CC2), U508.47 (C2_CC2)
- new net USBC2_CONN_RX1+: C510.1, J502.B11 (RX1+)
- new net USBC2_CONN_RX1-: C508.1, J502.B10 (RX1-)
- new net USBC2_CONN_RX2+: C518.1, J502.A11 (RX2+)
- new net USBC2_CONN_RX2-: C516.1, J502.A10 (RX2-)
- new net USBC2_CONN_TX1+: C514.1, J502.A2 (TX1+)
- new net USBC2_CONN_TX1-: C512.1, J502.A3 (TX1-)
- new net USBC2_CONN_TX2+: C522.1, J502.B2 (TX2+)
- new net USBC2_CONN_TX2-: C520.1, J502.B3 (TX2-)
- new net USBC2_DDCCLK: R508.1
- new net USBC2_DDCDAT: R509.1
- new net USBC2_SBU1: C532.2, C534.1, D511.2 (A2), J502.A8 (SBU1), R509.2
- new net USBC2_SBU2: C533.2, C535.1, D512.2 (A2), J502.B8 (SBU2), R508.2
- new net USBC2_TX0_D+: C514.2, U502.4, U502.7 (NC)
- new net USBC2_TX0_D-: C512.2, U502.5, U502.6 (NC)
- new net USBC2_TX1_D+: C522.2, U504.5, U504.6 (NC)
- new net USBC2_TX1_D-: C520.2, U504.4, U504.7 (NC)
- new net USBC2_TXRX0_D+: C510.2, U502.1, U502.10 (NC)
- new net USBC2_TXRX0_D-: C508.2, U502.2, U502.9 (NC)
- new net USBC2_TXRX1_D+: C518.2, U504.2, U504.9 (NC)
- new net USBC2_TXRX1_D-: C516.2, U504.1, U504.10 (NC)
- new net USBC2_USB2_D+: D509.2 (A2), J502.A6 (D+), J502.B6 (D+)
- new net USBC2_USB2_D-: D510.2 (A2), J502.A7 (D-), J502.B7 (D-)
- new net USBC2_VBUS: C502.1, J502.A4 (VBUS), J502.A9 (VBUS), J502.B4 (VBUS), J502.B9 (VBUS), U505.6 (OUT), U508.3 (VBUS2)
- new net VBAT: C602.2, C613.2, Q602.1 (S), Q602.2 (S), Q602.3 (S), R603.1, R612.1, R613.1, R614.1, TP601.1
- new net VBATSNS: C613.1, Q607.1 (D), Q607.2 (D), Q607.3 (D), R611.1, R613.2
- new net VBUS_5VIN: U505.5 (IN), U506.5 (IN)
- new net VCHARGE: C603.1, R601.1, R604.1, R609.1, TP602.1, U508.1 (PP_HV2), U508.11 (PP_HV1)
- new net VSYSTEM: C606.1, C607.1, C608.1, C609.1, Q604.5 (D), Q607.5 (S), TP603.1, U601.22 (VSYS)
- new net ~{PMCALERT}: U508.34 (~{I2C2_IRQ})
- no-connect marks 0 -> 30
Other:
- note added: "2.2 or 3.3 exactly"
- note added: "25mm connector spacing for PD debugger, 15 on macbook"
- note added: "Caution: non-standard pinout!"
- note added: "Cell count: 3s V(BATPRESZ) = 55% (52-65%) of REGN(6v) >500K total"
- note added: "DDC/SBU"
- note added: "Design for 800khz Fsw (default)"
- note added: "Drains are floating"
- note added: "ESD protection"
- note added: "PBI charges and discharges the cap"
- note added: "Port 1 -> 0x38 Port 2 -> 0x3F"
- note added: "Sense"
- note added: "Source power control"
- note added: "TODO: surface mount sensor?"
- note added: "These diodes are the wrong logic level"
- note added: "V(ILIM_HIZ) = 1 V + 40 × IDPM × RAC IDPM = max current e.g. 3A->2.2V, 1.5A->1.6V"
- note added: "default configuration: 1 (DFP + DP) (Rratio 0.1..0.18)"
